Commit message: Add new URDF-Model and the the implementation of the collision mechanism

File: data/objects/Winter/mmm.urdf (robot description, URDF)
Before this commit: robot unknown type, 126 links, 125 joints
Links:
- link BTSegment_joint: geometry collision mesh filename=models/collada/BTSegment_joint_visu.dae scale=1 1 1; visual mesh filename=models/collada/BTSegment_joint_visu.dae scale=1 1 1
- link BUNsegment_joint: geometry collision mesh filename=models/collada/BUNsegment_joint_visu.dae scale=1 1 1; visual mesh filename=models/collada/BUNsegment_joint_visu.dae scale=1 1 1
- link LAy_joint: geometry collision mesh filename=models/collada/LAy_joint_visu.dae scale=1 1 1; visual mesh filename=models/collada/LAy_joint_visu.dae scale=1 1 1
- link LEsegment_joint: geometry collision mesh filename=models/collada/LEsegment_joint_visu.dae scale=1 1 1; visual mesh filename=models/collada/LEsegment_joint_visu.dae scale=1 1 1
- link LFx_joint: geometry collision mesh filename=models/collada/LFx_joint_visu.dae scale=1 1 1; visual mesh filename=models/collada/LFx_joint_visu.dae scale=1 1 1
- link LHsegment_joint: geometry collision mesh filename=models/collada/LHsegment_joint_visu.dae scale=1 1 1; visual mesh filename=models/collada/LHsegment_joint_visu.dae scale=1 1 1
- link LKsegment_joint: geometry collision mesh filename=models/collada/LKsegment_joint_visu.dae scale=1 1 1; visual mesh filename=models/collada/LKsegment_joint_visu.dae scale=1 1 1

Commit message: correct the collision-tags

File: data/objects/Winter/mmm.urdf (robot description, URDF)
Before this commit: robot unknown type, 126 links, 125 joints
Links:
- link LAsegment_joint: geometry collision mesh filename=models/collada/LAsegment_joint_visu.dae scale=1 1 1; visual mesh filename=models/collada/LAsegment_joint_visu.dae scale=1 1 1
- link LMrot_joint: geometry collision mesh filename=models/collada/LMrot_joint_visu.dae scale=1 1 1; visual mesh filename=models/collada/LMrot_joint_visu.dae scale=1 1 1
- link LSCsegment_joint: geometry collision mesh filename=models/collada/LSCsegment_joint_visu.dae scale=1 1 1; visual mesh filename=models/collada/LSCsegment_joint_visu.dae scale=1 1 1
- link LSsegment_joint: geometry collision mesh filename=models/collada/LSsegment_joint_visu.dae scale=1 1 1; visual mesh filename=models/collada/LSsegment_joint_visu.dae scale=1 1 1
- link LWsegment_joint: geometry collision mesh filename=models/collada/LWsegment_joint_visu.dae scale=1 1 1; visual mesh filename=models/collada/LWsegment_joint_visu.dae scale=1 1 1
- link LWy_joint: geometry collision mesh filename=models/collada/LWy_joint_visu.dae scale=1 1 1; visual mesh filename=models/collada/LWy_joint_visu.dae scale=1 1 1
- link LeftEyeSegmentY_joint: geometry collision mesh filename=models/collada/LeftEyeSegmentY_joint_visu.dae scale=1 1 1; visual mesh filename=models/collada/LeftEyeSegmentY_joint_visu.dae scale=1 1 1
- link LeftFingerJoint11y_joint: geometry collision mesh filename=models/collada/LeftFingerJoint11y_joint_visu.dae scale=1 1 1; visual mesh filename=models/collada/LeftFingerJoint11y_joint_visu.dae scale=1 1 1
- link LeftFingerJoint12y_joint: geometry collision mesh filename=models/collada/LeftFingerJoint12y_joint_visu.dae scale=1 1 1; visual mesh filename=models/collada/LeftFingerJoint12y_joint_visu.dae scale=1 1 1
- link LeftFingerJoint13y_joint: geometry collision mesh filename=models/collada/LeftFingerJoint13y_joint_visu.dae scale=1 1 1; visual mesh filename=models/collada/LeftFingerJoint13y_joint_visu.dae scale=1 1 1
- link LeftFingerJoint21y_joint: geometry collision mesh filename=models/collada/LeftFingerJoint21y_joint_visu.dae scale=1 1 1; visual mesh filename=models/collada/LeftFingerJoint21y_joint_visu.dae scale=1 1 1
- link LeftFingerJoint22y_joint: geometry collision mesh filename=models/collada/LeftFingerJoint22y_joint_visu.dae scale=1 1 1; visual mesh filename=models/collada/LeftFingerJoint22y_joint_visu.dae scale=1 1 1
- link LeftFingerJoint23y_joint: geometry collision mesh filename=models/collada/LeftFingerJoint23y_joint_visu.dae scale=1 1 1; visual mesh filename=models/collada/LeftFingerJoint23y_joint_visu.dae scale=1 1 1
- link LeftFingerJoint31y_joint: geometry collision mesh filename=models/collada/LeftFingerJoint31y_joint_visu.dae scale=1 1 1; visual mesh filename=models/collada/LeftFingerJoint31y_joint_visu.dae scale=1 1 1
- link LeftFingerJoint32y_joint: geometry collision mesh filename=models/collada/LeftFingerJoint32y_joint_visu.dae scale=1 1 1; visual mesh filename=models/collada/LeftFingerJoint32y_joint_visu.dae scale=1 1 1
- link LeftFingerJoint33y_joint: geometry collision mesh filename=models/collada/LeftFingerJoint33y_joint_visu.dae scale=1 1 1; visual mesh filename=models/collada/LeftFingerJoint33y_joint_visu.dae scale=1 1 1
- link LeftFingerJoint40y_joint: geometry collision mesh filename=models/collada/LeftFingerJoint40y_joint_visu.dae scale=1 1 1; visual mesh filename=models/collada/LeftFingerJoint40y_joint_visu.dae scale=1 1 1
- link LeftFingerJoint41y_joint: geometry collision mesh filename=models/collada/LeftFingerJoint41y_joint_visu.dae scale=1 1 1; visual mesh filename=models/collada/LeftFingerJoint41y_joint_visu.dae scale=1 1 1
- link LeftFingerJoint42y_joint: geometry collision mesh filename=models/collada/LeftFingerJoint42y_joint_visu.dae scale=1 1 1; visual mesh filename=models/collada/LeftFingerJoint42y_joint_visu.dae scale=1 1 1
- link LeftFingerJoint43y_joint: geometry collision mesh filename=models/collada/LeftFingerJoint43y_joint_visu.dae scale=1 1 1; visual mesh filename=models/collada/LeftFingerJoint43y_joint_visu.dae scale=1 1 1
- link LeftFingerJoint50y_joint: geometry collision mesh filename=models/collada/LeftFingerJoint50y_joint_visu.dae scale=1 1 1; visual mesh filename=models/collada/LeftFingerJoint50y_joint_visu.dae scale=1 1 1
- link LeftFingerJoint51y_joint: geometry collision mesh filename=models/collada/LeftFingerJoint51y_joint_visu.dae scale=1 1 1; visual mesh filename=models/collada/LeftFingerJoint51y_joint_visu.dae scale=1 1 1
- link LeftFingerJoint52y_joint: geometry collision mesh filename=models/collada/LeftFingerJoint52y_joint_visu.dae scale=1 1 1; visual mesh filename=models/collada/LeftFingerJoint52y_joint_visu.dae scale=1 1 1
- link LeftFingerJoint53y_joint: geometry collision mesh filename=models/collada/LeftFingerJoint53y_joint_visu.dae scale=1 1 1; visual mesh filename=models/collada/LeftFingerJoint53y_joint_visu.dae scale=1 1 1
- link RAsegment_joint: geometry collision mesh filename=models/collada/RAsegment_joint_visu.dae scale=1 1 1; visual mesh filename=models/collada/RAsegment_joint_visu.dae scale=1 1 1
- link RAy_joint: geometry collision mesh filename=models/collada/RAy_joint_visu.dae scale=1 1 1; visual mesh filename=models/collada/RAy_joint_visu.dae scale=1 1 1
- link REsegment_joint: geometry collision mesh filename=models/collada/REsegment_joint_visu.dae scale=1 1 1; visual mesh filename=models/collada/REsegment_joint_visu.dae scale=1 1 1
- link RFx_joint: geometry collision mesh filename=models/collada/RFx_joint_visu.dae scale=1 1 1; visual mesh filename=models/collada/RFx_joint_visu.dae scale=1 1 1
- link RHsegment_joint: geometry collision mesh filename=models/collada/RHsegment_joint_visu.dae scale=1 1 1; visual mesh filename=models/collada/RHsegment_joint_visu.dae scale=1 1 1
- link RKsegment_joint: geometry collision mesh filename=models/collada/RKsegment_joint_visu.dae scale=1 1 1; visual mesh filename=models/collada/RKsegment_joint_visu.dae scale=1 1 1
- link RMrot_joint: geometry collision mesh filename=models/collada/RMrot_joint_visu.dae scale=1 1 1; visual mesh filename=models/collada/RMrot_joint_visu.dae scale=1 1 1
- link RSCsegment_joint: geometry collision mesh filename=models/collada/RSCsegment_joint_visu.dae scale=1 1 1; visual mesh filename=models/collada/RSCsegment_joint_visu.dae scale=1 1 1
- link RSsegment_joint: geometry collision mesh filename=models/collada/RSsegment_joint_visu.dae scale=1 1 1; visual mesh filename=models/collada/RSsegment_joint_visu.dae scale=1 1 1
- link RWsegment_joint: geometry collision mesh filename=models/collada/RWsegment_joint_visu.dae scale=1 1 1; visual mesh filename=models/collada/RWsegment_joint_visu.dae scale=1 1 1
- link RWy_joint: geometry collision mesh filename=models/collada/RWy_joint_visu.dae scale=1 1 1; visual mesh filename=models/collada/RWy_joint_visu.dae scale=1 1 1
- link RightEyeSegmentY_joint: geometry collision mesh filename=models/collada/RightEyeSegmentY_joint_visu.dae scale=1 1 1; visual mesh filename=models/collada/RightEyeSegmentY_joint_visu.dae scale=1 1 1
- link RightFingerJoint11y_joint: geometry collision mesh filename=models/collada/RightFingerJoint11y_joint_visu.dae scale=1 1 1; visual mesh filename=models/collada/RightFingerJoint11y_joint_visu.dae scale=1 1 1
- link RightFingerJoint12y_joint: geometry collision mesh filename=models/collada/RightFingerJoint12y_joint_visu.dae scale=1 1 1; visual mesh filename=models/collada/RightFingerJoint12y_joint_visu.dae scale=1 1 1
- link RightFingerJoint13y_joint: geometry collision mesh filename=models/collada/RightFingerJoint13y_joint_visu.dae scale=1 1 1; visual mesh filename=models/collada/RightFingerJoint13y_joint_visu.dae scale=1 1 1
- link RightFingerJoint21y_joint: geometry collision mesh filename=models/collada/RightFingerJoint21y_joint_visu.dae scale=1 1 1; visual mesh filename=models/collada/RightFingerJoint21y_joint_visu.dae scale=1 1 1
- link RightFingerJoint22y_joint: geometry collision mesh filename=models/collada/RightFingerJoint22y_joint_visu.dae scale=1 1 1; visual mesh filename=models/collada/RightFingerJoint22y_joint_visu.dae scale=1 1 1
- link RightFingerJoint23y_joint: geometry collision mesh filename=models/collada/RightFingerJoint23y_joint_visu.dae scale=1 1 1; visual mesh filename=models/collada/RightFingerJoint23y_joint_visu.dae scale=1 1 1
- link RightFingerJoint31y_joint: geometry collision mesh filename=models/collada/RightFingerJoint31y_joint_visu.dae scale=1 1 1; visual mesh filename=models/collada/RightFingerJoint31y_joint_visu.dae scale=1 1 1
- link RightFingerJoint32y_joint: geometry collision mesh filename=models/collada/RightFingerJoint32y_joint_visu.dae scale=1 1 1; visual mesh filename=models/collada/RightFingerJoint32y_joint_visu.dae scale=1 1 1
- link RightFingerJoint33y_joint: geometry collision mesh filename=models/collada/RightFingerJoint33y_joint_visu.dae scale=1 1 1; visual mesh filename=models/collada/RightFingerJoint33y_joint_visu.dae scale=1 1 1
- link RightFingerJoint40y_joint: geometry collision mesh filename=models/collada/RightFingerJoint40y_joint_visu.dae scale=1 1 1; visual mesh filename=models/collada/RightFingerJoint40y_joint_visu.dae scale=1 1 1
- link RightFingerJoint41y_joint: geometry collision mesh filename=models/collada/RightFingerJoint41y_joint_visu.dae scale=1 1 1; visual mesh filename=models/collada/RightFingerJoint41y_joint_visu.dae scale=1 1 1
- link RightFingerJoint42y_joint: geometry collision mesh filename=models/collada/RightFingerJoint42y_joint_visu.dae scale=1 1 1; visual mesh filename=models/collada/RightFingerJoint42y_joint_visu.dae scale=1 1 1
- link RightFingerJoint43y_joint: geometry collision mesh filename=models/collada/RightFingerJoint43y_joint_visu.dae scale=1 1 1; visual mesh filename=models/collada/RightFingerJoint43y_joint_visu.dae scale=1 1 1
- link RightFingerJoint50y_joint: geometry collision mesh filename=models/collada/RightFingerJoint50y_joint_visu.dae scale=1 1 1; visual mesh filename=models/collada/RightFingerJoint50y_joint_visu.dae scale=1 1 1
- link RightFingerJoint51y_joint: geometry collision mesh filename=models/collada/RightFingerJoint51y_joint_visu.dae scale=1 1 1; visual mesh filename=models/collada/RightFingerJoint51y_joint_visu.dae scale=1 1 1
- link RightFingerJoint52y_joint: geometry collision mesh filename=models/collada/RightFingerJoint52y_joint_visu.dae scale=1 1 1; visual mesh filename=models/collada/RightFingerJoint52y_joint_visu.dae scale=1 1 1
- link RightFingerJoint53y_joint: geometry collision mesh filename=models/collada/RightFingerJoint53y_joint_visu.dae scale=1 1 1; visual mesh filename=models/collada/RightFingerJoint53y_joint_visu.dae scale=1 1 1
