Commit message: Remove the root element mmm_modidied.urdf

File: data/objects/Winter/mmm_modified.urdf (robot description, URDF)
Before this commit: robot unknown type, 123 links, 123 joints
Links:
- added link MidHeadSegment_joint
Joints:
- joint LeftEyeSegmentX_joint: parent HeadSegment_joint -> MidHeadSegment_joint
- joint MidHeadSegment_joint: child HeadSegment_joint -> MidHeadSegment_joint
- joint RightEyeSegmentX_joint: parent HeadSegment_joint -> MidHeadSegment_joint

Commit message: Impelement the calcul of inertial-tensors for all meshes

File: data/objects/Winter/mmm_modified.urdf (robot description, URDF)
Before this commit: robot unknown type, 124 links, 123 joints
Links:
- link MidHeadSegment_joint: mass None -> 0.07; geometry collision mesh filename=models/collada/HeadSegment_joint_visu.dae scale=1 1 1; visual mesh filename=models/collada/HeadSegment_joint_visu.dae scale=1 1 1

Commit message: New implementation in mmm_modified.urdf

File: data/objects/Winter/mmm_modified.urdf (robot description, URDF)
Before this commit: robot unknown type, 124 links, 123 joints
Links:
- removed link BLNx_joint
- removed link BLNy_joint
- removed link BLNz_joint
- removed link BPSegment_joint
- removed link BPx_joint
- removed link BPy_joint
- removed link BPz_joint
- removed link BTSegment_joint
- removed link BTx_joint
- removed link BTy_joint
- removed link BTz_joint
- removed link BUNx_joint
- removed link BUNy_joint
- removed link BUNz_joint
- removed link HeadSegment_joint
- removed link LAx_joint
- removed link LAy_joint
- removed link LAz_joint
- removed link LEx_joint
- removed link LEz_joint
- removed link LHx_joint
- removed link LHy_joint
- removed link LHz_joint
- removed link LKx_joint
- removed link LSCx_joint
- removed link LSCy_joint
- removed link LSCz_joint
- removed link LSx_joint
- removed link LSy_joint
- removed link LSz_joint
- removed link LWx_joint
- removed link LWy_joint
- removed link LeftEyeSegmentX_joint
- removed link LeftEyeSegmentY_joint
- removed link LeftFingerJoint11y_joint
- removed link LeftFingerJoint11z_joint
- removed link LeftFingerJoint12y_joint
- removed link LeftFingerJoint13y_joint
- removed link LeftFingerJoint21x_joint
- removed link LeftFingerJoint21y_joint
- removed link LeftFingerJoint22y_joint
- removed link LeftFingerJoint23y_joint
- removed link LeftFingerJoint31x_joint
- removed link LeftFingerJoint31y_joint
- removed link LeftFingerJoint32y_joint
- removed link LeftFingerJoint33y_joint
- removed link LeftFingerJoint40y_joint
- removed link LeftFingerJoint41x_joint
- removed link LeftFingerJoint41y_joint
- removed link LeftFingerJoint42y_joint
- removed link LeftFingerJoint43y_joint
- removed link LeftFingerJoint50y_joint
- removed link LeftFingerJoint51x_joint
- removed link LeftFingerJoint51y_joint
- removed link LeftFingerJoint52y_joint
- removed link LeftFingerJoint53y_joint
- removed link LeftHandSegment_joint
- removed link MidHeadSegment_joint
- removed link RAx_joint
- removed link RAy_joint
- removed link RAz_joint
- removed link REx_joint
- removed link REz_joint
- removed link RFx_joint
- removed link RHx_joint
- removed link RHy_joint
- removed link RHz_joint
- removed link RKx_joint
- removed link RSCx_joint
- removed link RSCy_joint
- removed link RSCz_joint
- removed link RSx_joint
- removed link RSy_joint
- removed link RSz_joint
- removed link RWx_joint
- removed link RWy_joint
- removed link RightEyeSegmentX_joint
- removed link RightEyeSegmentY_joint
- removed link RightFingerJoint11y_joint
- removed link RightFingerJoint11z_joint
- removed link RightFingerJoint12y_joint
- removed link RightFingerJoint13y_joint
- removed link RightFingerJoint21x_joint
- removed link RightFingerJoint21y_joint
- removed link RightFingerJoint22y_joint
- removed link RightFingerJoint23y_joint
- removed link RightFingerJoint31x_joint
- removed link RightFingerJoint31y_joint
- removed link RightFingerJoint32y_joint
- removed link RightFingerJoint33y_joint
- removed link RightFingerJoint40y_joint
- removed link RightFingerJoint41x_joint
- removed link RightFingerJoint41y_joint
- removed link RightFingerJoint42y_joint
- removed link RightFingerJoint43y_joint
- removed link RightFingerJoint50y_joint
- removed link RightFingerJoint51x_joint
- removed link RightFingerJoint51y_joint
- removed link RightFingerJoint52y_joint
- removed link RightFingerJoint53y_joint
- removed link RightHandSegment_joint
- removed link collarSegment_joint
- added link BPsegment_joint, mass 0.11
- added link BTsegment_joint, mass 0.1; visual mesh filename=models/collada/BTSegment_joint_visu.dae scale=1 1 1
- added link Headsegment_joint, mass 0.07; visual mesh filename=models/collada/HeadSegment_joint_visu.dae scale=1 1 1
- added link LeftHandsegment_joint, mass 0.006
- added link MidHeadsegment_joint
- added link RFsegment_joint; visual mesh filename=models/collada/RFx_joint_visu.dae scale=1 1 1
- added link RightEyesegment_joint; visual mesh filename=models/collada/RightEyeSegmentY_joint_visu.dae scale=1 1 1
- added link RightFootLength_joint
- added link RightHandsegment_joint, mass 0.006
- added link collarsegment_joint, mass 0.17
- added link root
- link BLNsegment_joint: mass 0.11 -> None
- link BUNsegment_joint: geometry visual mesh filename=models/collada/BUNsegment_joint_visu.dae scale=1 1 1
- link LAsegment_joint: geometry visual mesh filename=models/collada/LAsegment_joint_visu.dae scale=1 1 1
- link LEsegment_joint: geometry visual mesh filename=models/collada/LEsegment_joint_visu.dae scale=1 1 1
- link LFx_joint: mass 0.027 -> None; geometry visual mesh filename=models/collada/LFx_joint_visu.dae scale=1 1 1
- link LHsegment_joint: geometry visual mesh filename=models/collada/LHsegment_joint_visu.dae scale=1 1 1
- link LKsegment_joint: geometry visual mesh filename=models/collada/LKsegment_joint_visu.dae scale=1 1 1
- link LMrot_joint: geometry visual mesh filename=models/collada/LMrot_joint_visu.dae scale=1 1 1
- link LSCsegment_joint: geometry visual mesh filename=models/collada/LSCsegment_joint_visu.dae scale=1 1 1
- link LSsegment_joint: geometry visual mesh filename=models/collada/LSsegment_joint_visu.dae scale=1 1 1
- link LWsegment_joint: geometry visual mesh filename=models/collada/LWsegment_joint_visu.dae scale=1 1 1
- link RAsegment_joint: geometry visual mesh filename=models/collada/RAsegment_joint_visu.dae scale=1 1 1
- link REsegment_joint: geometry visual mesh filename=models/collada/REsegment_joint_visu.dae scale=1 1 1
- link RHsegment_joint: geometry visual mesh filename=models/collada/RHsegment_joint_visu.dae scale=1 1 1
- link RKsegment_joint: geometry visual mesh filename=models/collada/RKsegment_joint_visu.dae scale=1 1 1
- link RMrot_joint: geometry visual mesh filename=models/collada/RMrot_joint_visu.dae scale=1 1 1
- link RSCsegment_joint: geometry visual mesh filename=models/collada/RSCsegment_joint_visu.dae scale=1 1 1
- link RSsegment_joint: geometry visual mesh filename=models/collada/RSsegment_joint_visu.dae scale=1 1 1
- link RWsegment_joint: geometry visual mesh filename=models/collada/RWsegment_joint_visu.dae scale=1 1 1
Joints:
- removed joint BLNsegment_joint
- removed joint BPSegment_joint
- removed joint BTSegment_joint
- removed joint BUNsegment_joint
- removed joint HeadSegment_joint
- removed joint LAsegment_joint
- removed joint LEsegment_joint
- removed joint LHsegment_joint
- removed joint LKsegment_joint
- removed joint LSCsegment_joint
- removed joint LSsegment_joint
- removed joint LWsegment_joint
- removed joint LeftEyeSegmentX_joint
- removed joint LeftEyeSegmentY_joint
- removed joint LeftFingerJoint11y_joint
- removed joint LeftFingerJoint11z_joint
- removed joint LeftFingerJoint12y_joint
- removed joint LeftFingerJoint13y_joint
- removed joint LeftFingerJoint21x_joint
- removed joint LeftFingerJoint21y_joint
- removed joint LeftFingerJoint22y_joint
- removed joint LeftFingerJoint23y_joint
- removed joint LeftFingerJoint31x_joint
- removed joint LeftFingerJoint31y_joint
- removed joint LeftFingerJoint32y_joint
- removed joint LeftFingerJoint33y_joint
- removed joint LeftFingerJoint40y_joint
- removed joint LeftFingerJoint41x_joint
- removed joint LeftFingerJoint41y_joint
- removed joint LeftFingerJoint42y_joint
- removed joint LeftFingerJoint43y_joint
- removed joint LeftFingerJoint50y_joint
- removed joint LeftFingerJoint51x_joint
- removed joint LeftFingerJoint51y_joint
- removed joint LeftFingerJoint52y_joint
- removed joint LeftFingerJoint53y_joint
- removed joint LeftHandSegment_joint
- removed joint MidHeadSegment_joint
- removed joint RAsegment_joint
- removed joint REsegment_joint
- removed joint RKsegment_joint
- removed joint RSCsegment_joint
- removed joint RSsegment_joint
- removed joint RWsegment_joint
- removed joint RightEyeSegmentX_joint
- removed joint RightEyeSegmentY_joint
- removed joint RightFingerJoint11y_joint
- removed joint RightFingerJoint11z_joint
- removed joint RightFingerJoint12y_joint
- removed joint RightFingerJoint13y_joint
- removed joint RightFingerJoint21x_joint
- removed joint RightFingerJoint21y_joint
- removed joint RightFingerJoint22y_joint
- removed joint RightFingerJoint23y_joint
- removed joint RightFingerJoint31x_joint
- removed joint RightFingerJoint31y_joint
- removed joint RightFingerJoint32y_joint
- removed joint RightFingerJoint33y_joint
- removed joint RightFingerJoint40y_joint
- removed joint RightFingerJoint41x_joint
- removed joint RightFingerJoint41y_joint
- removed joint RightFingerJoint42y_joint
- removed joint RightFingerJoint43y_joint
- removed joint RightFingerJoint50y_joint
- removed joint RightFingerJoint51x_joint
- removed joint RightFingerJoint51y_joint
- removed joint RightFingerJoint52y_joint
- removed joint RightFingerJoint53y_joint
- removed joint RightHandSegment_joint
- removed joint collarSegment_joint
- added joint Headsegment_joint: type fixed, parent BUNsegment_joint, child Headsegment_joint, origin xyz=0 0 0.13 rpy=0 -0 0
- added joint LeftHandsegment_joint: type fixed, parent LWsegment_joint, child LeftHandsegment_joint, origin xyz=0 0 -0.108 rpy=0 -0 0
- added joint MidHeadsegment_joint: type fixed, parent BUNsegment_joint, child MidHeadsegment_joint, origin xyz=0 0 0.066 rpy=0 -0 0
- added joint RightEyesegment_joint: type fixed, parent MidHeadsegment_joint, child RightEyesegment_joint, origin xyz=0.015 0 0 rpy=0 -0 0
- added joint RightFootLength_joint: type fixed, parent RightFootHeight_joint, child RightFootLength_joint, origin xyz=0 0.068 0 rpy=0 -0 0
- added joint RightHandsegment_joint: type fixed, parent RWsegment_joint, child RightHandsegment_joint, origin xyz=0 0 -0.108 rpy=0 -0 0
- added joint collarsegment_joint: type fixed, parent BTsegment_joint, child collarsegment_joint, origin xyz=0 0 0.188 rpy=0 -0 0
- added joint root_joint: type revolute, parent root, child root_joint, axis 0 0 1, limit lower=0 upper=0 effort=100 velocity=1
- joint BLNx_joint: axis 1 0 0 -> (none); child BLNx_joint -> BLNsegment_joint; origin (none) -> xyz=0 0 0.022 rpy=0 -0 0; parent BLNsegment_joint -> collarsegment_joint
- joint BLNy_joint: axis 0 1 0 -> (none); child BLNy_joint -> BLNsegment_joint; origin (none) -> xyz=0 0 0.022 rpy=0 -0 0; parent BLNz_joint -> collarsegment_joint
- joint BLNz_joint: axis 0 0 1 -> (none); child BLNz_joint -> BLNsegment_joint; origin (none) -> xyz=0 0 0.022 rpy=0 -0 0; parent BLNx_joint -> collarsegment_joint
- joint BPx_joint: axis 1 0 0 -> (none); child BPx_joint -> BPsegment_joint; parent BPSegment_joint -> root_joint
- joint BPy_joint: axis 0 1 0 -> (none); child BPy_joint -> BPsegment_joint; origin (none) -> xyz=0 0 0.04 rpy=0 -0 0; parent BPz_joint -> root_joint
- joint BPz_joint: axis 0 0 1 -> (none); child BPz_joint -> BPsegment_joint; origin (none) -> xyz=0 0 0.04 rpy=0 -0 0; parent BPx_joint -> root_joint
- joint BTx_joint: axis 1 0 0 -> (none); child BTx_joint -> BTsegment_joint; origin (none) -> xyz=0 0 0.06 rpy=0 -0 0; parent BTSegment_joint -> BPsegment_joint
- joint BTy_joint: axis 0 1 0 -> (none); child BTy_joint -> BTsegment_joint; origin (none) -> xyz=0 0 0.06 rpy=0 -0 0; parent BTz_joint -> BPsegment_joint
- joint BTz_joint: axis 0 0 1 -> (none); child BTz_joint -> BTsegment_joint; origin (none) -> xyz=0 0 0.06 rpy=0 -0 0; parent BTx_joint -> BPsegment_joint
- joint BUNx_joint: axis 1 0 0 -> (none); child BUNx_joint -> BUNsegment_joint; origin (none) -> xyz=0 0 0.03 rpy=0 -0 0; parent BUNsegment_joint -> BLNsegment_joint
- joint BUNy_joint: axis 0 1 0 -> (none); child BUNy_joint -> BUNsegment_joint; origin (none) -> xyz=0 0 0.03 rpy=0 -0 0; parent BUNz_joint -> BLNsegment_joint
- joint BUNz_joint: axis 0 0 1 -> (none); child BUNz_joint -> BUNsegment_joint; origin (none) -> xyz=0 0 0.03 rpy=0 -0 0; parent BUNx_joint -> BLNsegment_joint
- joint LAx_joint: axis 1 0 0 -> (none); child LAx_joint -> LAsegment_joint; origin (none) -> xyz=0 0 -0.246 rpy=0 -0 0
- joint LAy_joint: axis 0 1 0 -> (none); child LAy_joint -> LAsegment_joint; origin (none) -> xyz=0 0 -0.246 rpy=0 -0 0; parent LAz_joint -> LKsegment_joint
- joint LAz_joint: axis 0 0 1 -> (none); child LAz_joint -> LAsegment_joint; origin (none) -> xyz=0 0 -0.246 rpy=0 -0 0; parent LAx_joint -> LKsegment_joint
- joint LEx_joint: axis 1 0 0 -> (none); child LEx_joint -> LEsegment_joint; origin (none) -> xyz=0 0 -0.188 rpy=0 -0 0; parent LEsegment_joint -> LSsegment_joint
- joint LEz_joint: axis 0 0 1 -> (none); child LEz_joint -> LEsegment_joint; origin (none) -> xyz=0 0 -0.188 rpy=0 -0 0; parent LEx_joint -> LSsegment_joint
- joint LFx_joint: axis 1 0 0 -> (none)
- joint LHx_joint: axis 1 0 0 -> (none); child LHx_joint -> LHsegment_joint; origin (none) -> xyz=-0.052 0 0 rpy=0 -0 0; parent LHsegment_joint -> root_joint
- joint LHy_joint: axis 0 1 0 -> (none); child LHy_joint -> LHsegment_joint; origin (none) -> xyz=-0.052 0 0 rpy=0 -0 0; parent LHz_joint -> root_joint
- joint LHz_joint: axis 0 0 1 -> (none); child LHz_joint -> LHsegment_joint; origin (none) -> xyz=-0.052 0 0 rpy=0 -0 0; parent LHx_joint -> root_joint
- joint LKx_joint: axis 1 0 0 -> (none); child LKx_joint -> LKsegment_joint; origin (none) -> xyz=0 0 -0.245 rpy=0 -0 0; parent LKsegment_joint -> LHsegment_joint
- joint LMrot_joint: parent LAy_joint -> LAsegment_joint
- joint LSCx_joint: axis 1 0 0 -> (none); child LSCx_joint -> LSCsegment_joint; origin (none) -> xyz=-0.087 0 0 rpy=0 -0 0; parent LSCsegment_joint -> collarsegment_joint
- joint LSCy_joint: axis 0 1 0 -> (none); child LSCy_joint -> LSCsegment_joint; origin (none) -> xyz=-0.087 0 0 rpy=0 -0 0; parent LSCz_joint -> collarsegment_joint
- joint LSCz_joint: axis 0 0 1 -> (none); child LSCz_joint -> LSCsegment_joint; origin (none) -> xyz=-0.087 0 0 rpy=0 -0 0; parent LSCx_joint -> collarsegment_joint
- joint LSx_joint: axis 1 0 0 -> (none); child LSx_joint -> LSsegment_joint; origin (none) -> xyz=-0.023 0 0 rpy=0 -0 0; parent LSsegment_joint -> LSCsegment_joint
- joint LSy_joint: axis 0 1 0 -> (none); child LSy_joint -> LSsegment_joint; origin (none) -> xyz=-0.023 0 0 rpy=0 -0 0; parent LSz_joint -> LSCsegment_joint
- joint LSz_joint: axis 0 0 1 -> (none); child LSz_joint -> LSsegment_joint; origin (none) -> xyz=-0.023 0 0 rpy=0 -0 0; parent LSx_joint -> LSCsegment_joint
- joint LWx_joint: axis 1 0 0 -> (none); child LWx_joint -> LWsegment_joint; origin (none) -> xyz=0 0 -0.145 rpy=0 -0 0; parent LWsegment_joint -> LEsegment_joint
- joint LWy_joint: axis 0 1 0 -> (none); child LWy_joint -> LWsegment_joint; origin (none) -> xyz=0 0 -0.145 rpy=0 -0 0; parent LWx_joint -> LEsegment_joint
- joint LeftFootHeight_joint: parent LAy_joint -> LAsegment_joint
- joint RAx_joint: axis 1 0 0 -> (none); child RAx_joint -> RAsegment_joint; origin (none) -> xyz=0 0 -0.246 rpy=0 -0 0; parent RAsegment_joint -> RKsegment_joint
- joint RAy_joint: axis 0 1 0 -> (none); child RAy_joint -> RAsegment_joint; origin (none) -> xyz=0 0 -0.246 rpy=0 -0 0; parent RAz_joint -> RKsegment_joint
- joint RAz_joint: axis 0 0 1 -> (none); child RAz_joint -> RAsegment_joint; origin (none) -> xyz=0 0 -0.246 rpy=0 -0 0; parent RAx_joint -> RKsegment_joint
- joint REx_joint: axis 1 0 0 -> (none); child REx_joint -> REsegment_joint; origin (none) -> xyz=0 0 -0.188 rpy=0 -0 0; parent REsegment_joint -> RSsegment_joint
- joint REz_joint: axis 0 0 1 -> (none); child REz_joint -> REsegment_joint; origin (none) -> xyz=0 0 -0.188 rpy=0 -0 0; parent REx_joint -> RSsegment_joint
- joint RFx_joint: axis 1 0 0 -> (none); child RFx_joint -> RFsegment_joint
- joint RHx_joint: axis 0 1 0 -> (none); child RHx_joint -> RHsegment_joint; origin (none) -> xyz=0.052 0 0 rpy=0 -0 0; parent RHsegment_joint -> root_joint
- joint RHy_joint: axis 1 0 0 -> (none); child RHy_joint -> RHsegment_joint; origin (none) -> xyz=0.052 0 0 rpy=0 -0 0; parent RHz_joint -> root_joint
- joint RHz_joint: axis 0 0 1 -> (none); child RHz_joint -> RHsegment_joint; origin (none) -> xyz=0.052 0 0 rpy=0 -0 0; parent RHx_joint -> root_joint
- joint RKx_joint: axis 1 0 0 -> (none); child RKx_joint -> RKsegment_joint; origin (none) -> xyz=0 0 -0.245 rpy=0 -0 0; parent RKsegment_joint -> RHsegment_joint
- joint RMrot_joint: parent RAy_joint -> RAsegment_joint
- joint RSCx_joint: axis 1 0 0 -> (none); child RSCx_joint -> RSCsegment_joint; origin (none) -> xyz=0.087 0 0 rpy=0 -0 0; parent RSCsegment_joint -> collarsegment_joint
- joint RSCy_joint: axis 0 1 0 -> (none); child RSCy_joint -> RSCsegment_joint; origin (none) -> xyz=0.087 0 0 rpy=0 -0 0; parent RSCz_joint -> collarsegment_joint
- joint RSCz_joint: axis 0 0 1 -> (none); child RSCz_joint -> RSCsegment_joint; origin (none) -> xyz=0.087 0 0 rpy=0 -0 0; parent RSCx_joint -> collarsegment_joint
- joint RSx_joint: axis 1 0 0 -> (none); child RSx_joint -> RSsegment_joint; origin (none) -> xyz=0.023 0 0 rpy=0 -0 0; parent RSsegment_joint -> RSCsegment_joint
- joint RSy_joint: axis 0 1 0 -> (none); child RSy_joint -> RSsegment_joint; origin (none) -> xyz=0.023 0 0 rpy=0 -0 0; parent RSz_joint -> RSCsegment_joint
- joint RSz_joint: axis 0 0 1 -> (none); child RSz_joint -> RSsegment_joint; origin (none) -> xyz=0.023 0 0 rpy=0 -0 0; parent RSx_joint -> RSCsegment_joint
- joint RWx_joint: axis 1 0 0 -> (none); child RWx_joint -> RWsegment_joint; origin (none) -> xyz=0 0 -0.145 rpy=0 -0 0; parent RWsegment_joint -> REsegment_joint
- joint RWy_joint: axis 0 1 0 -> (none); child RWy_joint -> RWsegment_joint; origin (none) -> xyz=0 0 -0.145 rpy=0 -0 0; parent RWx_joint -> REsegment_joint
- joint RightFootHeight_joint: parent RAy_joint -> RAsegment_joint
