Commit message: New robot.urdf file

File: data/objects/robot.urdf (robot description, URDF)
Before this commit: robot dumpUrdf, 16 links, 15 joints
Links:
- removed link base
- removed link chest
- removed link left_ankle
- removed link left_elbow
- removed link left_hip
- removed link left_knee
- removed link left_shoulder
- removed link left_wrist
- removed link neck
- removed link right_ankle
- removed link right_elbow
- removed link right_hip
- removed link right_knee
- removed link right_shoulder
- removed link right_wrist
- removed link root
- added link Head, mass 2.2392; collision sphere radius=0.089005; visual sphere radius=0.089005
- added link Head_f1, mass 0
- added link Head_f2, mass 0
- added link L3, mass 6.3444; collision box size=0.13815 0.16323 0.085916; visual box size=0.13815 0.16323 0.085916
- added link L3_f1, mass 0
- added link L3_f2, mass 0
- added link L5, mass 6.3444; collision box size=0.13815 0.16323 0.095104; visual box size=0.13815 0.16323 0.095104
- added link L5_f1, mass 0
- added link L5_f2, mass 0
- added link LeftFoot, mass 0.8086; collision box size=0.17983 0.074775 0.078509; visual box size=0.17983 0.074775 0.078509
- added link LeftFoot_f1, mass 0
- added link LeftFoot_f2, mass 0
- added link LeftForeArm, mass 1.244; collision cylinder length=0.22247 radius=0.019633; visual cylinder length=0.22247 radius=0.019633
- added link LeftForeArm_f1, mass 0
- added link LeftForeArm_f2, mass 0
- added link LeftHand, mass 0.3732; collision box size=0.11145 0.16718 0.039266; visual box size=0.11145 0.16718 0.039266
- added link LeftHand_f1, mass 0
- added link LeftHand_f2, mass 0
- added link LeftLowerLeg, mass 2.2703; collision cylinder length=0.40608 radius=0.037388; visual cylinder length=0.40608 radius=0.037388
- added link LeftLowerLeg_f1, mass 0
- added link LeftLowerLeg_f2, mass 0
- added link LeftShoulder, mass 1.9282; collision cylinder length=0.13047 radius=0.023574; visual cylinder length=0.13047 radius=0.023574
- added link LeftShoulder_f1, mass 0
- added link LeftShoulder_f2, mass 0
- added link LeftToe, mass 0.0933; collision box size=0.060173 0.074775 0.014191; visual box size=0.060173 0.074775 0.014191
- added link LeftToe_f1, mass 0
- added link LeftToe_f2, mass 0
- added link LeftUpperArm, mass 1.866; collision cylinder length=0.26994 radius=0.029449; visual cylinder length=0.26994 radius=0.029449
- added link LeftUpperArm_f1, mass 0
- added link LeftUpperArm_f2, mass 0
- added link LeftUpperLeg, mass 7.775; collision cylinder length=0.44898 radius=0.0565; visual cylinder length=0.44898 radius=0.0565
- added link LeftUpperLeg_f1, mass 0
- added link LeftUpperLeg_f2, mass 0
- added link Neck, mass 0.7464; collision cylinder length=0.089252 radius=0.014205; visual cylinder length=0.089252 radius=0.014205
- added link Neck_f1, mass 0
- added link Neck_f2, mass 0
- added link Pelvis, mass 4.976; collision box size=0.13815 0.24914 0.097469; visual box size=0.13815 0.24914 0.097469
- added link RightFoot, mass 0.8086; collision box size=0.17983 0.074775 0.078509; visual box size=0.17983 0.074775 0.078509
- added link RightFoot_f1, mass 0
- added link RightFoot_f2, mass 0
- added link RightForeArm, mass 1.244; collision cylinder length=0.22247 radius=0.019633; visual cylinder length=0.22247 radius=0.019633
- added link RightForeArm_f1, mass 0
- added link RightForeArm_f2, mass 0
- added link RightHand, mass 0.3732; collision box size=0.11145 0.16718 0.039266; visual box size=0.11145 0.16718 0.039266
- added link RightHand_f1, mass 0
- added link RightHand_f2, mass 0
- added link RightLowerLeg, mass 2.2703; collision cylinder length=0.40608 radius=0.037388; visual cylinder length=0.40608 radius=0.037388
- added link RightLowerLeg_f1, mass 0
- added link RightLowerLeg_f2, mass 0
- added link RightShoulder, mass 1.9282; collision cylinder length=0.13047 radius=0.023574; visual cylinder length=0.13047 radius=0.023574
- added link RightShoulder_f1, mass 0
- added link RightShoulder_f2, mass 0
- added link RightToe, mass 0.0933; collision box size=0.060173 0.074775 0.014191; visual box size=0.060173 0.074775 0.014191
- added link RightToe_f1, mass 0
- added link RightToe_f2, mass 0
- added link RightUpperArm, mass 1.866; collision cylinder length=0.26994 radius=0.029449; visual cylinder length=0.26994 radius=0.029449
- added link RightUpperArm_f1, mass 0
- added link RightUpperArm_f2, mass 0
- added link RightUpperLeg, mass 7.775; collision cylinder length=0.44898 radius=0.0565; visual cylinder length=0.44898 radius=0.0565
- added link RightUpperLeg_f1, mass 0
- added link RightUpperLeg_f2, mass 0
- added link T12, mass 6.3444; collision box size=0.13815 0.16323 0.085916; visual box size=0.13815 0.16323 0.085916
- added link T12_f1, mass 0
- added link T12_f2, mass 0
- added link T8, mass 2.488; collision box size=0.13457 0.052626 0.11975; visual box size=0.13457 0.052626 0.11975
- added link T8_f1, mass 0
- added link T8_f2, mass 0
Joints:
- removed joint chest
- removed joint left_ankle
- removed joint left_elbow
- removed joint left_hip
- removed joint left_knee
- removed joint left_shoulder
- removed joint left_wrist
- removed joint neck
- removed joint right_ankle
- removed joint right_elbow
- removed joint right_hip
- removed joint right_knee
- removed joint right_shoulder
- removed joint right_wrist
- removed joint root
- added joint jC1Head_rotx: type revolute, parent Neck, child Head_f1, origin xyz=0.000152           0    0.089252 rpy=0 0 0, axis 1 0 0, limit lower=-10.0 upper=10.0 effort=30 velocity=1.0
- added joint jC1Head_roty: type revolute, parent Head_f1, child Head_f2, origin xyz=0 0 0 rpy=0 0 0, axis 0 1 0, limit lower=-10.0 upper=10.0 effort=30 velocity=1.0
- added joint jC1Head_rotz: type revolute, parent Head_f2, child Head, origin xyz=0 0 0 rpy=0 0 0, axis 0 0 1, limit lower=-10.0 upper=10.0 effort=30 velocity=1.0
- added joint jL1T12_rotx: type revolute, parent L3, child T12_f1, origin xyz=0           0    0.085916 rpy=0 0 0, axis 1 0 0, limit lower=-10.0 upper=10.0 effort=30 velocity=1.0
- added joint jL1T12_roty: type revolute, parent T12_f1, child T12_f2, origin xyz=0 0 0 rpy=0 0 0, axis 0 1 0, limit lower=-10.0 upper=10.0 effort=30 velocity=1.0
- added joint jL1T12_rotz: type revolute, parent T12_f2, child T12, origin xyz=0 0 0 rpy=0 0 0, axis 0 0 1, limit lower=-10.0 upper=10.0 effort=30 velocity=1.0
- added joint jL4L3_rotx: type revolute, parent L5, child L3_f1, origin xyz=0.000374           0    0.095104 rpy=0 0 0, axis 1 0 0, limit lower=-10.0 upper=10.0 effort=30 velocity=1.0
- added joint jL4L3_roty: type revolute, parent L3_f1, child L3_f2, origin xyz=0 0 0 rpy=0 0 0, axis 0 1 0, limit lower=-10.0 upper=10.0 effort=30 velocity=1.0
- added joint jL4L3_rotz: type revolute, parent L3_f2, child L3, origin xyz=0 0 0 rpy=0 0 0, axis 0 0 1, limit lower=-10.0 upper=10.0 effort=30 velocity=1.0
- added joint jL5S1_rotx: type revolute, parent Pelvis, child L5_f1, origin xyz=-0.000206           0    0.098478 rpy=0 0 0, axis 1 0 0, limit lower=-10.0 upper=10.0 effort=30 velocity=1.0
- added joint jL5S1_roty: type revolute, parent L5_f1, child L5_f2, origin xyz=0 0 0 rpy=0 0 0, axis 0 1 0, limit lower=-10.0 upper=10.0 effort=30 velocity=1.0
- added joint jL5S1_rotz: type revolute, parent L5_f2, child L5, origin xyz=0 0 0 rpy=0 0 0, axis 0 0 1, limit lower=-10.0 upper=10.0 effort=30 velocity=1.0
- added joint jLeftAnkle_rotx: type revolute, parent LeftLowerLeg, child LeftFoot_f1, origin xyz=0.000205           0    -0.40608 rpy=0 0 0, axis 1 0 0, limit lower=-10.0 upper=10.0 effort=30 velocity=1.0
- added joint jLeftAnkle_roty: type revolute, parent LeftFoot_f1, child LeftFoot_f2, origin xyz=0 0 0 rpy=0 0 0, axis 0 1 0, limit lower=-10.0 upper=10.0 effort=30 velocity=1.0
- added joint jLeftAnkle_rotz: type revolute, parent LeftFoot_f2, child LeftFoot, origin xyz=0 0 0 rpy=0 0 0, axis 0 0 1, limit lower=-10.0 upper=10.0 effort=30 velocity=1.0
- added joint jLeftBallFoot_rotx: type revolute, parent LeftFoot, child LeftToe_f1, origin xyz=0.14456           0   -0.064752 rpy=0 0 0, axis 1 0 0, limit lower=-10.0 upper=10.0 effort=30 velocity=1.0
- added joint jLeftBallFoot_roty: type revolute, parent LeftToe_f1, child LeftToe_f2, origin xyz=0 0 0 rpy=0 0 0, axis 0 1 0, limit lower=-10.0 upper=10.0 effort=30 velocity=1.0
- added joint jLeftBallFoot_rotz: type revolute, parent LeftToe_f2, child LeftToe, origin xyz=0 0 0 rpy=0 0 0, axis 0 0 1, limit lower=-10.0 upper=10.0 effort=30 velocity=1.0
- added joint jLeftC7Shoulder_rotx: type revolute, parent T8, child LeftShoulder_f1, origin xyz=0    0.026313    0.067052 rpy=0 0 0, axis 1 0 0, limit lower=-10.0 upper=10.0 effort=30 velocity=1.0
- added joint jLeftC7Shoulder_roty: type revolute, parent LeftShoulder_f1, child LeftShoulder_f2, origin xyz=0 0 0 rpy=0 0 0, axis 0 1 0, limit lower=-10.0 upper=10.0 effort=30 velocity=1.0
- added joint jLeftC7Shoulder_rotz: type revolute, parent LeftShoulder_f2, child LeftShoulder, origin xyz=0 0 0 rpy=0 0 0, axis 0 0 1, limit lower=-10.0 upper=10.0 effort=30 velocity=1.0
- added joint jLeftElbow_rotx: type revolute, parent LeftUpperArm, child LeftForeArm_f1, origin xyz=0     0.26994           0 rpy=0 0 0, axis 1 0 0, limit lower=-10.0 upper=10.0 effort=30 velocity=1.0
- added joint jLeftElbow_roty: type revolute, parent LeftForeArm_f1, child LeftForeArm_f2, origin xyz=0 0 0 rpy=0 0 0, axis 0 1 0, limit lower=-10.0 upper=10.0 effort=30 velocity=1.0
- added joint jLeftElbow_rotz: type revolute, parent LeftForeArm_f2, child LeftForeArm, origin xyz=0 0 0 rpy=0 0 0, axis 0 0 1, limit lower=-10.0 upper=10.0 effort=30 velocity=1.0
- added joint jLeftHip_rotx: type revolute, parent Pelvis, child LeftUpperLeg_f1, origin xyz=0.000103    0.081614    0.001009 rpy=0 0 0, axis 1 0 0, limit lower=-10.0 upper=10.0 effort=30 velocity=1.0
- added joint jLeftHip_roty: type revolute, parent LeftUpperLeg_f1, child LeftUpperLeg_f2, origin xyz=0 0 0 rpy=0 0 0, axis 0 1 0, limit lower=-10.0 upper=10.0 effort=30 velocity=1.0
- added joint jLeftHip_rotz: type revolute, parent LeftUpperLeg_f2, child LeftUpperLeg, origin xyz=0 0 0 rpy=0 0 0, axis 0 0 1, limit lower=-10.0 upper=10.0 effort=30 velocity=1.0
- added joint jLeftKnee_rotx: type revolute, parent LeftUpperLeg, child LeftLowerLeg_f1, origin xyz=3.6e-05           0    -0.44898 rpy=0 0 0, axis 1 0 0, limit lower=-10.0 upper=10.0 effort=30 velocity=1.0
- added joint jLeftKnee_roty: type revolute, parent LeftLowerLeg_f1, child LeftLowerLeg_f2, origin xyz=0 0 0 rpy=0 0 0, axis 0 1 0, limit lower=-10.0 upper=10.0 effort=30 velocity=1.0
- added joint jLeftKnee_rotz: type revolute, parent LeftLowerLeg_f2, child LeftLowerLeg, origin xyz=0 0 0 rpy=0 0 0, axis 0 0 1, limit lower=-10.0 upper=10.0 effort=30 velocity=1.0
- added joint jLeftShoulder_rotx: type revolute, parent LeftShoulder, child LeftUpperArm_f1, origin xyz=0     0.13047           0 rpy=0 0 0, axis 1 0 0, limit lower=-10.0 upper=10.0 effort=30 velocity=1.0
- added joint jLeftShoulder_roty: type revolute, parent LeftUpperArm_f1, child LeftUpperArm_f2, origin xyz=0 0 0 rpy=0 0 0, axis 0 1 0, limit lower=-10.0 upper=10.0 effort=30 velocity=1.0
- added joint jLeftShoulder_rotz: type revolute, parent LeftUpperArm_f2, child LeftUpperArm, origin xyz=0 0 0 rpy=0 0 0, axis 0 0 1, limit lower=-10.0 upper=10.0 effort=30 velocity=1.0
- added joint jLeftWrist_rotx: type revolute, parent LeftForeArm, child LeftHand_f1, origin xyz=7.7e-05     0.22247           0 rpy=0 0 0, axis 1 0 0, limit lower=-10.0 upper=10.0 effort=30 velocity=1.0
- added joint jLeftWrist_roty: type revolute, parent LeftHand_f1, child LeftHand_f2, origin xyz=0 0 0 rpy=0 0 0, axis 0 1 0, limit lower=-10.0 upper=10.0 effort=30 velocity=1.0
- added joint jLeftWrist_rotz: type revolute, parent LeftHand_f2, child LeftHand, origin xyz=0 0 0 rpy=0 0 0, axis 0 0 1, limit lower=-10.0 upper=10.0 effort=30 velocity=1.0
- added joint jRightAnkle_rotx: type revolute, parent RightLowerLeg, child RightFoot_f1, origin xyz=0.000205           0    -0.40608 rpy=0 0 0, axis 1 0 0, limit lower=-10.0 upper=10.0 effort=30 velocity=1.0
- added joint jRightAnkle_roty: type revolute, parent RightFoot_f1, child RightFoot_f2, origin xyz=0 0 0 rpy=0 0 0, axis 0 1 0, limit lower=-10.0 upper=10.0 effort=30 velocity=1.0
- added joint jRightAnkle_rotz: type revolute, parent RightFoot_f2, child RightFoot, origin xyz=0 0 0 rpy=0 0 0, axis 0 0 1, limit lower=-10.0 upper=10.0 effort=30 velocity=1.0
- added joint jRightBallFoot_rotx: type revolute, parent RightFoot, child RightToe_f1, origin xyz=0.14456           0   -0.064752 rpy=0 0 0, axis 1 0 0, limit lower=-10.0 upper=10.0 effort=30 velocity=1.0
- added joint jRightBallFoot_roty: type revolute, parent RightToe_f1, child RightToe_f2, origin xyz=0 0 0 rpy=0 0 0, axis 0 1 0, limit lower=-10.0 upper=10.0 effort=30 velocity=1.0
- added joint jRightBallFoot_rotz: type revolute, parent RightToe_f2, child RightToe, origin xyz=0 0 0 rpy=0 0 0, axis 0 0 1, limit lower=-10.0 upper=10.0 effort=30 velocity=1.0
- added joint jRightC7Shoulder_rotx: type revolute, parent T8, child RightShoulder_f1, origin xyz=0   -0.026313    0.067052 rpy=0 0 0, axis 1 0 0, limit lower=-10.0 upper=10.0 effort=30 velocity=1.0
- added joint jRightC7Shoulder_roty: type revolute, parent RightShoulder_f1, child RightShoulder_f2, origin xyz=0 0 0 rpy=0 0 0, axis 0 1 0, limit lower=-10.0 upper=10.0 effort=30 velocity=1.0
- added joint jRightC7Shoulder_rotz: type revolute, parent RightShoulder_f2, child RightShoulder, origin xyz=0 0 0 rpy=0 0 0, axis 0 0 1, limit lower=-10.0 upper=10.0 effort=30 velocity=1.0
- added joint jRightElbow_rotx: type revolute, parent RightUpperArm, child RightForeArm_f1, origin xyz=0    -0.26994           0 rpy=0 0 0, axis 1 0 0, limit lower=-10.0 upper=10.0 effort=30 velocity=1.0
- added joint jRightElbow_roty: type revolute, parent RightForeArm_f1, child RightForeArm_f2, origin xyz=0 0 0 rpy=0 0 0, axis 0 1 0, limit lower=-10.0 upper=10.0 effort=30 velocity=1.0
- added joint jRightElbow_rotz: type revolute, parent RightForeArm_f2, child RightForeArm, origin xyz=0 0 0 rpy=0 0 0, axis 0 0 1, limit lower=-10.0 upper=10.0 effort=30 velocity=1.0
- added joint jRightHip_rotx: type revolute, parent Pelvis, child RightUpperLeg_f1, origin xyz=0.000103   -0.081614    0.001009 rpy=0 0 0, axis 1 0 0, limit lower=-10.0 upper=10.0 effort=30 velocity=1.0
- added joint jRightHip_roty: type revolute, parent RightUpperLeg_f1, child RightUpperLeg_f2, origin xyz=0 0 0 rpy=0 0 0, axis 0 1 0, limit lower=-10.0 upper=10.0 effort=30 velocity=1.0
- added joint jRightHip_rotz: type revolute, parent RightUpperLeg_f2, child RightUpperLeg, origin xyz=0 0 0 rpy=0 0 0, axis 0 0 1, limit lower=-10.0 upper=10.0 effort=30 velocity=1.0
- added joint jRightKnee_rotx: type revolute, parent RightUpperLeg, child RightLowerLeg_f1, origin xyz=3.6e-05           0    -0.44898 rpy=0 0 0, axis 1 0 0, limit lower=-10.0 upper=10.0 effort=30 velocity=1.0
- added joint jRightKnee_roty: type revolute, parent RightLowerLeg_f1, child RightLowerLeg_f2, origin xyz=0 0 0 rpy=0 0 0, axis 0 1 0, limit lower=-10.0 upper=10.0 effort=30 velocity=1.0
- added joint jRightKnee_rotz: type revolute, parent RightLowerLeg_f2, child RightLowerLeg, origin xyz=0 0 0 rpy=0 0 0, axis 0 0 1, limit lower=-10.0 upper=10.0 effort=30 velocity=1.0
- added joint jRightShoulder_rotx: type revolute, parent RightShoulder, child RightUpperArm_f1, origin xyz=0    -0.13047           0 rpy=0 0 0, axis 1 0 0, limit lower=-10.0 upper=10.0 effort=30 velocity=1.0
- added joint jRightShoulder_roty: type revolute, parent RightUpperArm_f1, child RightUpperArm_f2, origin xyz=0 0 0 rpy=0 0 0, axis 0 1 0, limit lower=-10.0 upper=10.0 effort=30 velocity=1.0
- added joint jRightShoulder_rotz: type revolute, parent RightUpperArm_f2, child RightUpperArm, origin xyz=0 0 0 rpy=0 0 0, axis 0 0 1, limit lower=-10.0 upper=10.0 effort=30 velocity=1.0
- added joint jRightWrist_rotx: type revolute, parent RightForeArm, child RightHand_f1, origin xyz=7.7e-05    -0.22247           0 rpy=0 0 0, axis 1 0 0, limit lower=-10.0 upper=10.0 effort=30 velocity=1.0
- added joint jRightWrist_roty: type revolute, parent RightHand_f1, child RightHand_f2, origin xyz=0 0 0 rpy=0 0 0, axis 0 1 0, limit lower=-10.0 upper=10.0 effort=30 velocity=1.0
- added joint jRightWrist_rotz: type revolute, parent RightHand_f2, child RightHand, origin xyz=0 0 0 rpy=0 0 0, axis 0 0 1, limit lower=-10.0 upper=10.0 effort=30 velocity=1.0
- added joint jT1C7_rotx: type revolute, parent T8, child Neck_f1, origin xyz=0           0     0.11975 rpy=0 0 0, axis 1 0 0, limit lower=-10.0 upper=10.0 effort=30 velocity=1.0
- added joint jT1C7_roty: type revolute, parent Neck_f1, child Neck_f2, origin xyz=0 0 0 rpy=0 0 0, axis 0 1 0, limit lower=-10.0 upper=10.0 effort=30 velocity=1.0
- added joint jT1C7_rotz: type revolute, parent Neck_f2, child Neck, origin xyz=0 0 0 rpy=0 0 0, axis 0 0 1, limit lower=-10.0 upper=10.0 effort=30 velocity=1.0
- added joint jT9T8_rotx: type revolute, parent T12, child T8_f1, origin xyz=0           0    0.085916 rpy=0 0 0, axis 1 0 0, limit lower=-10.0 upper=10.0 effort=30 velocity=1.0
- added joint jT9T8_roty: type revolute, parent T8_f1, child T8_f2, origin xyz=0 0 0 rpy=0 0 0, axis 0 1 0, limit lower=-10.0 upper=10.0 effort=30 velocity=1.0
- added joint jT9T8_rotz: type revolute, parent T8_f2, child T8, origin xyz=0 0 0 rpy=0 0 0, axis 0 0 1, limit lower=-10.0 upper=10.0 effort=30 velocity=1.0

Commit message: Add motions to the simulation

File: data/objects/robot.urdf (robot description, URDF)
Before this commit: robot XSensStyleModel_template, 67 links, 66 joints
Links:
- link Head: mass 2.2392 -> 3
- link L3: mass 6.3444 -> 7
- link L5: mass 6.3444 -> 7
- link LeftFoot: mass 0.8086 -> 1
- link LeftForeArm: mass 1.244 -> 2
- link LeftHand: mass 0.3732 -> 1
- link LeftLowerLeg: mass 2.2703 -> 3
- link LeftShoulder: mass 1.9282 -> 2
- link LeftUpperArm: mass 1.866 -> 2
- link LeftUpperLeg: mass 7.775 -> 7
- link Neck: mass 0.7464 -> 1
- link Pelvis: mass 4.976 -> 2
- link RightFoot: mass 0.8086 -> 1
- link RightForeArm: mass 1.244 -> 2
- link RightHand: mass 0.3732 -> 1
- link RightLowerLeg: mass 2.2703 -> 3
- link RightShoulder: mass 1.9282 -> 3
- link RightUpperArm: mass 1.866 -> 2
- link RightUpperLeg: mass 7.775 -> 7
- link T12: mass 6.3444 -> 7
- link T8: mass 2.488 -> 3
