Commit message: Add names of joints partially conform to mmm-notation and clean up the motion-dataset extraction

File: data/objects/robot.urdf (robot description, URDF)
Before this commit: robot XSensStyleModel_template, 67 links, 66 joints
Joints:
- removed joint jC1Head_rotx
- removed joint jC1Head_roty
- removed joint jC1Head_rotz
- removed joint jL5S1_rotx
- removed joint jL5S1_roty
- removed joint jL5S1_rotz
- removed joint jLeftAnkle_rotx
- removed joint jLeftAnkle_roty
- removed joint jLeftAnkle_rotz
- removed joint jLeftBallFoot_rotx
- removed joint jLeftBallFoot_roty
- removed joint jLeftBallFoot_rotz
- removed joint jLeftC7Shoulder_rotx
- removed joint jLeftC7Shoulder_roty
- removed joint jLeftC7Shoulder_rotz
- removed joint jLeftElbow_rotx
- removed joint jLeftElbow_roty
- removed joint jLeftElbow_rotz
- removed joint jLeftHip_rotx
- removed joint jLeftHip_roty
- removed joint jLeftHip_rotz
- removed joint jLeftKnee_rotx
- removed joint jLeftKnee_roty
- removed joint jLeftKnee_rotz
- removed joint jLeftShoulder_rotx
- removed joint jLeftShoulder_roty
- removed joint jLeftShoulder_rotz
- removed joint jLeftWrist_rotx
- removed joint jLeftWrist_roty
- removed joint jLeftWrist_rotz
- removed joint jRightAnkle_rotx
- removed joint jRightAnkle_roty
- removed joint jRightAnkle_rotz
- removed joint jRightBallFoot_rotx
- removed joint jRightBallFoot_roty
- removed joint jRightBallFoot_rotz
- removed joint jRightC7Shoulder_rotx
- removed joint jRightC7Shoulder_roty
- removed joint jRightC7Shoulder_rotz
- removed joint jRightElbow_rotx
- removed joint jRightElbow_roty
- removed joint jRightElbow_rotz
- removed joint jRightHip_rotx
- removed joint jRightHip_roty
- removed joint jRightHip_rotz
- removed joint jRightKnee_rotx
- removed joint jRightKnee_roty
- removed joint jRightKnee_rotz
- removed joint jRightShoulder_rotx
- removed joint jRightShoulder_roty
- removed joint jRightShoulder_rotz
- removed joint jRightWrist_rotx
- removed joint jRightWrist_roty
- removed joint jRightWrist_rotz
- removed joint jT1C7_rotx
- removed joint jT1C7_roty
- removed joint jT1C7_rotz
- added joint BLNx_joint: type revolute, parent T8, child Neck_f1, origin xyz=0           0     0.11975 rpy=0 0 0, axis 1 0 0, limit lower=-10.0 upper=10.0 effort=30 velocity=1.0
- added joint BLNy_joint: type revolute, parent Neck_f1, child Neck_f2, origin xyz=0 0 0 rpy=0 0 0, axis 0 1 0, limit lower=-10.0 upper=10.0 effort=30 velocity=1.0
- added joint BLNz_joint: type revolute, parent Neck_f2, child Neck, origin xyz=0 0 0 rpy=0 0 0, axis 0 0 1, limit lower=-10.0 upper=10.0 effort=30 velocity=1.0
- added joint BTx_joint: type revolute, parent Pelvis, child L5_f1, origin xyz=-0.000206           0    0.098478 rpy=0 0 0, axis 1 0 0, limit lower=-10.0 upper=10.0 effort=30 velocity=1.0
- added joint BTy_joint: type revolute, parent L5_f1, child L5_f2, origin xyz=0 0 0 rpy=0 0 0, axis 0 1 0, limit lower=-10.0 upper=10.0 effort=30 velocity=1.0
- added joint BTz_joint: type revolute, parent L5_f2, child L5, origin xyz=0 0 0 rpy=0 0 0, axis 0 0 1, limit lower=-10.0 upper=10.0 effort=30 velocity=1.0
- added joint BUNx_joint: type revolute, parent Neck, child Head_f1, origin xyz=0.000152           0    0.089252 rpy=0 0 0, axis 1 0 0, limit lower=-10.0 upper=10.0 effort=30 velocity=1.0
- added joint BUNy_joint: type revolute, parent Head_f1, child Head_f2, origin xyz=0 0 0 rpy=0 0 0, axis 0 1 0, limit lower=-10.0 upper=10.0 effort=30 velocity=1.0
- added joint BUNz_joint: type revolute, parent Head_f2, child Head, origin xyz=0 0 0 rpy=0 0 0, axis 0 0 1, limit lower=-10.0 upper=10.0 effort=30 velocity=1.0
- added joint LAx_joint: type revolute, parent LeftLowerLeg, child LeftFoot_f1, origin xyz=0.000205           0    -0.40608 rpy=0 0 0, axis 1 0 0, limit lower=-10.0 upper=10.0 effort=30 velocity=1.0
- added joint LAy_joint: type revolute, parent LeftFoot_f1, child LeftFoot_f2, origin xyz=0 0 0 rpy=0 0 0, axis 0 1 0, limit lower=-10.0 upper=10.0 effort=30 velocity=1.0
- added joint LAz_joint: type revolute, parent LeftFoot_f2, child LeftFoot, origin xyz=0 0 0 rpy=0 0 0, axis 0 0 1, limit lower=-10.0 upper=10.0 effort=30 velocity=1.0
- added joint LEx_joint: type revolute, parent LeftUpperArm, child LeftForeArm_f1, origin xyz=0     0.26994           0 rpy=0 0 0, axis 1 0 0, limit lower=-10.0 upper=10.0 effort=30 velocity=1.0
- added joint LEy_joint: type revolute, parent LeftForeArm_f1, child LeftForeArm_f2, origin xyz=0 0 0 rpy=0 0 0, axis 0 1 0, limit lower=-10.0 upper=10.0 effort=30 velocity=1.0
- added joint LEz_joint: type revolute, parent LeftForeArm_f2, child LeftForeArm, origin xyz=0 0 0 rpy=0 0 0, axis 0 0 1, limit lower=-10.0 upper=10.0 effort=30 velocity=1.0
- added joint LFx_joint: type revolute, parent LeftFoot, child LeftToe_f1, origin xyz=0.14456           0   -0.064752 rpy=0 0 0, axis 1 0 0, limit lower=-10.0 upper=10.0 effort=30 velocity=1.0
- added joint LFy_joint: type revolute, parent LeftToe_f1, child LeftToe_f2, origin xyz=0 0 0 rpy=0 0 0, axis 0 1 0, limit lower=-10.0 upper=10.0 effort=30 velocity=1.0
- added joint LFz_joint: type revolute, parent LeftToe_f2, child LeftToe, origin xyz=0 0 0 rpy=0 0 0, axis 0 0 1, limit lower=-10.0 upper=10.0 effort=30 velocity=1.0
- added joint LHx_joint: type revolute, parent Pelvis, child LeftUpperLeg_f1, origin xyz=0.000103    0.081614    0.001009 rpy=0 0 0, axis 1 0 0, limit lower=-10.0 upper=10.0 effort=30 velocity=1.0
- added joint LHy_joint: type revolute, parent LeftUpperLeg_f1, child LeftUpperLeg_f2, origin xyz=0 0 0 rpy=0 0 0, axis 0 1 0, limit lower=-10.0 upper=10.0 effort=30 velocity=1.0
- added joint LHz_joint: type revolute, parent LeftUpperLeg_f2, child LeftUpperLeg, origin xyz=0 0 0 rpy=0 0 0, axis 0 0 1, limit lower=-10.0 upper=10.0 effort=30 velocity=1.0
- added joint LKx_joint: type revolute, parent LeftUpperLeg, child LeftLowerLeg_f1, origin xyz=3.6e-05           0    -0.44898 rpy=0 0 0, axis 1 0 0, limit lower=-10.0 upper=10.0 effort=30 velocity=1.0
- added joint LKy_joint: type revolute, parent LeftLowerLeg_f1, child LeftLowerLeg_f2, origin xyz=0 0 0 rpy=0 0 0, axis 0 1 0, limit lower=-10.0 upper=10.0 effort=30 velocity=1.0
- added joint LKz_joint: type revolute, parent LeftLowerLeg_f2, child LeftLowerLeg, origin xyz=0 0 0 rpy=0 0 0, axis 0 0 1, limit lower=-10.0 upper=10.0 effort=30 velocity=1.0
- added joint LSCx_joint: type revolute, parent T8, child LeftShoulder_f1, origin xyz=0    0.026313    0.067052 rpy=0 0 0, axis 1 0 0, limit lower=-10.0 upper=10.0 effort=30 velocity=1.0
- added joint LSCy_joint: type revolute, parent LeftShoulder_f1, child LeftShoulder_f2, origin xyz=0 0 0 rpy=0 0 0, axis 0 1 0, limit lower=-10.0 upper=10.0 effort=30 velocity=1.0
- added joint LSCz_joint: type revolute, parent LeftShoulder_f2, child LeftShoulder, origin xyz=0 0 0 rpy=0 0 0, axis 0 0 1, limit lower=-10.0 upper=10.0 effort=30 velocity=1.0
- added joint LSx_joint: type revolute, parent LeftShoulder, child LeftUpperArm_f1, origin xyz=0     0.13047           0 rpy=0 0 0, axis 1 0 0, limit lower=-10.0 upper=10.0 effort=30 velocity=1.0
- added joint LSy_joint: type revolute, parent LeftUpperArm_f1, child LeftUpperArm_f2, origin xyz=0 0 0 rpy=0 0 0, axis 0 1 0, limit lower=-10.0 upper=10.0 effort=30 velocity=1.0
- added joint LSz_joint: type revolute, parent LeftUpperArm_f2, child LeftUpperArm, origin xyz=0 0 0 rpy=0 0 0, axis 0 0 1, limit lower=-10.0 upper=10.0 effort=30 velocity=1.0
- added joint LWx_joint: type revolute, parent LeftForeArm, child LeftHand_f1, origin xyz=7.7e-05     0.22247           0 rpy=0 0 0, axis 1 0 0, limit lower=-10.0 upper=10.0 effort=30 velocity=1.0
- added joint LWy_joint: type revolute, parent LeftHand_f1, child LeftHand_f2, origin xyz=0 0 0 rpy=0 0 0, axis 0 1 0, limit lower=-10.0 upper=10.0 effort=30 velocity=1.0
- added joint LWz_joint: type revolute, parent LeftHand_f2, child LeftHand, origin xyz=0 0 0 rpy=0 0 0, axis 0 0 1, limit lower=-10.0 upper=10.0 effort=30 velocity=1.0
- added joint RAx_joint: type revolute, parent RightLowerLeg, child RightFoot_f1, origin xyz=0.000205           0    -0.40608 rpy=0 0 0, axis 1 0 0, limit lower=-10.0 upper=10.0 effort=30 velocity=1.0
- added joint RAy_joint: type revolute, parent RightFoot_f1, child RightFoot_f2, origin xyz=0 0 0 rpy=0 0 0, axis 0 1 0, limit lower=-10.0 upper=10.0 effort=30 velocity=1.0
- added joint RAz_joint: type revolute, parent RightFoot_f2, child RightFoot, origin xyz=0 0 0 rpy=0 0 0, axis 0 0 1, limit lower=-10.0 upper=10.0 effort=30 velocity=1.0
- added joint REx_joint: type revolute, parent RightUpperArm, child RightForeArm_f1, origin xyz=0    -0.26994           0 rpy=0 0 0, axis 1 0 0, limit lower=-10.0 upper=10.0 effort=30 velocity=1.0
- added joint REy_joint: type revolute, parent RightForeArm_f1, child RightForeArm_f2, origin xyz=0 0 0 rpy=0 0 0, axis 0 1 0, limit lower=-10.0 upper=10.0 effort=30 velocity=1.0
- added joint REz_joint: type revolute, parent RightForeArm_f2, child RightForeArm, origin xyz=0 0 0 rpy=0 0 0, axis 0 0 1, limit lower=-10.0 upper=10.0 effort=30 velocity=1.0
- added joint RFx_joint: type revolute, parent RightFoot, child RightToe_f1, origin xyz=0.14456           0   -0.064752 rpy=0 0 0, axis 1 0 0, limit lower=-10.0 upper=10.0 effort=30 velocity=1.0
- added joint RFy_joint: type revolute, parent RightToe_f1, child RightToe_f2, origin xyz=0 0 0 rpy=0 0 0, axis 0 1 0, limit lower=-10.0 upper=10.0 effort=30 velocity=1.0
- added joint RFz_joint: type revolute, parent RightToe_f2, child RightToe, origin xyz=0 0 0 rpy=0 0 0, axis 0 0 1, limit lower=-10.0 upper=10.0 effort=30 velocity=1.0
- added joint RHx_joint: type revolute, parent Pelvis, child RightUpperLeg_f1, origin xyz=0.000103   -0.081614    0.001009 rpy=0 0 0, axis 1 0 0, limit lower=-10.0 upper=10.0 effort=30 velocity=1.0
- added joint RHy_joint: type revolute, parent RightUpperLeg_f1, child RightUpperLeg_f2, origin xyz=0 0 0 rpy=0 0 0, axis 0 1 0, limit lower=-10.0 upper=10.0 effort=30 velocity=1.0
- added joint RHz_joint: type revolute, parent RightUpperLeg_f2, child RightUpperLeg, origin xyz=0 0 0 rpy=0 0 0, axis 0 0 1, limit lower=-10.0 upper=10.0 effort=30 velocity=1.0
- added joint RKx_joint: type revolute, parent RightUpperLeg, child RightLowerLeg_f1, origin xyz=3.6e-05           0    -0.44898 rpy=0 0 0, axis 1 0 0, limit lower=-10.0 upper=10.0 effort=30 velocity=1.0
- added joint RKy_joint: type revolute, parent RightLowerLeg_f1, child RightLowerLeg_f2, origin xyz=0 0 0 rpy=0 0 0, axis 0 1 0, limit lower=-10.0 upper=10.0 effort=30 velocity=1.0
- added joint RKz_joint: type revolute, parent RightLowerLeg_f2, child RightLowerLeg, origin xyz=0 0 0 rpy=0 0 0, axis 0 0 1, limit lower=-10.0 upper=10.0 effort=30 velocity=1.0
- added joint RSCx_joint: type revolute, parent T8, child RightShoulder_f1, origin xyz=0   -0.026313    0.067052 rpy=0 0 0, axis 1 0 0, limit lower=-10.0 upper=10.0 effort=30 velocity=1.0
- added joint RSCy_joint: type revolute, parent RightShoulder_f1, child RightShoulder_f2, origin xyz=0 0 0 rpy=0 0 0, axis 0 1 0, limit lower=-10.0 upper=10.0 effort=30 velocity=1.0
- added joint RSCz_joint: type revolute, parent RightShoulder_f2, child RightShoulder, origin xyz=0 0 0 rpy=0 0 0, axis 0 0 1, limit lower=-10.0 upper=10.0 effort=30 velocity=1.0
- added joint RSx_joint: type revolute, parent RightShoulder, child RightUpperArm_f1, origin xyz=0    -0.13047           0 rpy=0 0 0, axis 1 0 0, limit lower=-10.0 upper=10.0 effort=30 velocity=1.0
- added joint RSy_joint: type revolute, parent RightUpperArm_f1, child RightUpperArm_f2, origin xyz=0 0 0 rpy=0 0 0, axis 0 1 0, limit lower=-10.0 upper=10.0 effort=30 velocity=1.0
- added joint RSz_joint: type revolute, parent RightUpperArm_f2, child RightUpperArm, origin xyz=0 0 0 rpy=0 0 0, axis 0 0 1, limit lower=-10.0 upper=10.0 effort=30 velocity=1.0
- added joint RWx_joint: type revolute, parent RightForeArm, child RightHand_f1, origin xyz=7.7e-05    -0.22247           0 rpy=0 0 0, axis 1 0 0, limit lower=-10.0 upper=10.0 effort=30 velocity=1.0
- added joint RWy_joint: type revolute, parent RightHand_f1, child RightHand_f2, origin xyz=0 0 0 rpy=0 0 0, axis 0 1 0, limit lower=-10.0 upper=10.0 effort=30 velocity=1.0
- added joint RWz_joint: type revolute, parent RightHand_f2, child RightHand, origin xyz=0 0 0 rpy=0 0 0, axis 0 0 1, limit lower=-10.0 upper=10.0 effort=30 velocity=1.0
