Commit message: Add Frame class to dataset to extract all the informations about joints

File: data/objects/robot.urdf (robot description, URDF)
Before this commit: robot unknown type, 126 links, 125 joints
Links:
- removed link BLNsegment_joint
- removed link BLNx_joint
- removed link BLNy_joint
- removed link BLNz_joint
- removed link BPSegment_joint
- removed link BPx_joint
- removed link BPy_joint
- removed link BPz_joint
- removed link BTSegment_joint
- removed link BTx_joint
- removed link BTy_joint
- removed link BTz_joint
- removed link BUNsegment_joint
- removed link BUNx_joint
- removed link BUNy_joint
- removed link BUNz_joint
- removed link HeadSegment_joint
- removed link LAsegment_joint
- removed link LAx_joint
- removed link LAy_joint
- removed link LAz_joint
- removed link LEsegment_joint
- removed link LEx_joint
- removed link LEz_joint
- removed link LFx_joint
- removed link LHsegment_joint
- removed link LHx_joint
- removed link LHy_joint
- removed link LHz_joint
- removed link LKsegment_joint
- removed link LKx_joint
- removed link LMrot_joint
- removed link LSCsegment_joint
- removed link LSCx_joint
- removed link LSCy_joint
- removed link LSCz_joint
- removed link LSsegment_joint
- removed link LSx_joint
- removed link LSy_joint
- removed link LSz_joint
- removed link LWsegment_joint
- removed link LWx_joint
- removed link LWy_joint
- removed link LeftEyeSegmentX_joint
- removed link LeftEyeSegmentY_joint
- removed link LeftFingerJoint11y_joint
- removed link LeftFingerJoint11z_joint
- removed link LeftFingerJoint12y_joint
- removed link LeftFingerJoint13y_joint
- removed link LeftFingerJoint21x_joint
- removed link LeftFingerJoint21y_joint
- removed link LeftFingerJoint22y_joint
- removed link LeftFingerJoint23y_joint
- removed link LeftFingerJoint31x_joint
- removed link LeftFingerJoint31y_joint
- removed link LeftFingerJoint32y_joint
- removed link LeftFingerJoint33y_joint
- removed link LeftFingerJoint40y_joint
- removed link LeftFingerJoint41x_joint
- removed link LeftFingerJoint41y_joint
- removed link LeftFingerJoint42y_joint
- removed link LeftFingerJoint43y_joint
- removed link LeftFingerJoint50y_joint
- removed link LeftFingerJoint51x_joint
- removed link LeftFingerJoint51y_joint
- removed link LeftFingerJoint52y_joint
- removed link LeftFingerJoint53y_joint
- removed link LeftFootHeight_joint
- removed link LeftHandSegment_joint
- removed link MidHeadSegment_joint
- removed link RAsegment_joint
- removed link RAx_joint
- removed link RAy_joint
- removed link RAz_joint
- removed link REsegment_joint
- removed link REx_joint
- removed link REz_joint
- removed link RFx_joint
- removed link RHsegment_joint
- removed link RHx_joint
- removed link RHy_joint
- removed link RHz_joint
- removed link RKsegment_joint
- removed link RKx_joint
- removed link RMrot_joint
- removed link RSCsegment_joint
- removed link RSCx_joint
- removed link RSCy_joint
- removed link RSCz_joint
- removed link RSsegment_joint
- removed link RSx_joint
- removed link RSy_joint
- removed link RSz_joint
- removed link RWsegment_joint
- removed link RWx_joint
- removed link RWy_joint
- removed link RightEyeSegmentX_joint
- removed link RightEyeSegmentY_joint
- removed link RightFingerJoint11y_joint
- removed link RightFingerJoint11z_joint
- removed link RightFingerJoint12y_joint
- removed link RightFingerJoint13y_joint
- removed link RightFingerJoint21x_joint
- removed link RightFingerJoint21y_joint
- removed link RightFingerJoint22y_joint
- removed link RightFingerJoint23y_joint
- removed link RightFingerJoint31x_joint
- removed link RightFingerJoint31y_joint
- removed link RightFingerJoint32y_joint
- removed link RightFingerJoint33y_joint
- removed link RightFingerJoint40y_joint
- removed link RightFingerJoint41x_joint
- removed link RightFingerJoint41y_joint
- removed link RightFingerJoint42y_joint
- removed link RightFingerJoint43y_joint
- removed link RightFingerJoint50y_joint
- removed link RightFingerJoint51x_joint
- removed link RightFingerJoint51y_joint
- removed link RightFingerJoint52y_joint
- removed link RightFingerJoint53y_joint
- removed link RightFootHeight_joint
- removed link RightFootLength_joint
- removed link RightHandSegment_joint
- removed link collarSegment_joint
- removed link root
- removed link root_joint
- added link left_foot, mass 1.13114; collision capsule length=0.21095 radius=0.02700; collision capsule length=0.21095 radius=0.02700
- added link left_lower_arm, mass 1.22954; collision capsule length=0.27713 radius=0.03100; collision sphere radius=0.04000
- added link left_shin, mass 2.75570; collision capsule length=0.30000 radius=0.04900
- added link left_thigh, mass 4.75175; collision capsule length=0.34015 radius=0.06000
- added link left_upper_arm, mass 1.66108; collision capsule length=0.27713 radius=0.04000
- added link link1_11, mass 0.00000
- added link link1_13, mass 0.00000
- added link link1_14, mass 0.00000
- added link link1_16, mass 0.00000
- added link link1_17, mass 0.00000
- added link link1_18, mass 0.00000
- added link link1_2, mass 0.00000
- added link link1_20, mass 0.00000
- added link link1_22, mass 0.00000
- added link link1_23, mass 0.00000
- added link link1_25, mass 0.00000
- added link link1_26, mass 0.00000
- added link link1_28, mass 0.00000
- added link link1_3, mass 0.00000
- added link link1_30, mass 0.00000
- added link link1_31, mass 0.00000
- added link link1_33, mass 0.00000
- added link link1_5, mass 0.00000
- added link link1_7, mass 0.00000
- added link link1_8, mass 0.00000
- added link link1_9, mass 0.00000
- added link lwaist, mass 2.26195; collision capsule length=0.12000 radius=0.06000
- added link pelvis, mass 6.61619; collision capsule length=0.14000 radius=0.09000
- added link right_foot, mass 1.13114; collision capsule length=0.21095 radius=0.02700; collision capsule length=0.21095 radius=0.02700
- added link right_lower_arm, mass 1.22954; collision capsule length=0.27713 radius=0.03100; collision sphere radius=0.04000
- added link right_shin, mass 2.75570; collision capsule length=0.30000 radius=0.04900
- added link right_thigh, mass 4.75175; collision capsule length=0.34015 radius=0.06000
- added link right_upper_arm, mass 1.66108; collision capsule length=0.27713 radius=0.04000
- added link torso, mass 8.90746; collision capsule length=0.12000 radius=0.06000; collision capsule length=0.14000 radius=0.07000
Joints:
- removed joint BLNsegment_joint
- removed joint BLNx_joint
- removed joint BLNy_joint
- removed joint BLNz_joint
- removed joint BPSegment_joint
- removed joint BPx_joint
- removed joint BPy_joint
- removed joint BPz_joint
- removed joint BTSegment_joint
- removed joint BTx_joint
- removed joint BUNsegment_joint
- removed joint BUNx_joint
- removed joint BUNy_joint
- removed joint BUNz_joint
- removed joint HeadSegment_joint
- removed joint LAsegment_joint
- removed joint LAx_joint
- removed joint LAy_joint
- removed joint LAz_joint
- removed joint LEsegment_joint
- removed joint LEx_joint
- removed joint LEz_joint
- removed joint LFx_joint
- removed joint LHsegment_joint
- removed joint LHx_joint
- removed joint LHy_joint
- removed joint LHz_joint
- removed joint LKsegment_joint
- removed joint LKx_joint
- removed joint LMrot_joint
- removed joint LSCsegment_joint
- removed joint LSCx_joint
- removed joint LSCy_joint
- removed joint LSCz_joint
- removed joint LSsegment_joint
- removed joint LSx_joint
- removed joint LSy_joint
- removed joint LSz_joint
- removed joint LWsegment_joint
- removed joint LWx_joint
- removed joint LWy_joint
- removed joint LeftEyeSegmentX_joint
- removed joint LeftEyeSegmentY_joint
- removed joint LeftFingerJoint11y_joint
- removed joint LeftFingerJoint11z_joint
- removed joint LeftFingerJoint12y_joint
- removed joint LeftFingerJoint13y_joint
- removed joint LeftFingerJoint21x_joint
- removed joint LeftFingerJoint21y_joint
- removed joint LeftFingerJoint22y_joint
- removed joint LeftFingerJoint23y_joint
- removed joint LeftFingerJoint31x_joint
- removed joint LeftFingerJoint31y_joint
- removed joint LeftFingerJoint32y_joint
- removed joint LeftFingerJoint33y_joint
- removed joint LeftFingerJoint40y_joint
- removed joint LeftFingerJoint41x_joint
- removed joint LeftFingerJoint41y_joint
- removed joint LeftFingerJoint42y_joint
- removed joint LeftFingerJoint43y_joint
- removed joint LeftFingerJoint50y_joint
- removed joint LeftFingerJoint51x_joint
- removed joint LeftFingerJoint51y_joint
- removed joint LeftFingerJoint52y_joint
- removed joint LeftFingerJoint53y_joint
- removed joint LeftFootHeight_joint
- removed joint LeftHandSegment_joint
- removed joint MidHeadSegment_joint
- removed joint RAsegment_joint
- removed joint RAx_joint
- removed joint RAy_joint
- removed joint RAz_joint
- removed joint REsegment_joint
- removed joint REx_joint
- removed joint REz_joint
- removed joint RFx_joint
- removed joint RHsegment_joint
- removed joint RHx_joint
- removed joint RHy_joint
- removed joint RHz_joint
- removed joint RKsegment_joint
- removed joint RKx_joint
- removed joint RMrot_joint
- removed joint RSCsegment_joint
- removed joint RSCx_joint
- removed joint RSCy_joint
- removed joint RSCz_joint
- removed joint RSsegment_joint
- removed joint RSx_joint
- removed joint RSy_joint
- removed joint RSz_joint
- removed joint RWsegment_joint
- removed joint RWx_joint
- removed joint RWy_joint
- removed joint RightEyeSegmentX_joint
- removed joint RightEyeSegmentY_joint
- removed joint RightFingerJoint11y_joint
- removed joint RightFingerJoint11z_joint
- removed joint RightFingerJoint12y_joint
- removed joint RightFingerJoint13y_joint
- removed joint RightFingerJoint21x_joint
- removed joint RightFingerJoint21y_joint
- removed joint RightFingerJoint22y_joint
- removed joint RightFingerJoint23y_joint
- removed joint RightFingerJoint31x_joint
- removed joint RightFingerJoint31y_joint
- removed joint RightFingerJoint32y_joint
- removed joint RightFingerJoint33y_joint
- removed joint RightFingerJoint40y_joint
- removed joint RightFingerJoint41x_joint
- removed joint RightFingerJoint41y_joint
- removed joint RightFingerJoint42y_joint
- removed joint RightFingerJoint43y_joint
- removed joint RightFingerJoint50y_joint
- removed joint RightFingerJoint51x_joint
- removed joint RightFingerJoint51y_joint
- removed joint RightFingerJoint52y_joint
- removed joint RightFingerJoint53y_joint
- removed joint RightFootHeight_joint
- removed joint RightFootLength_joint
- removed joint RightHandSegment_joint
- removed joint collarSegment_joint
- removed joint root_joint
- added joint abdomen_x: type continuous, parent lwaist, child link1_5, origin xyz=-0.00040 0.00000 -0.06500 rpy=0.00000 -0.00400 0.00000, axis 1.00000 0.00000 0.00000
- added joint jointfix_0_14: type fixed, parent link1_14, child right_foot, origin xyz=0.00000 0.00000 -0.08000 rpy=0.00000 -0.00000 0.00000, axis 0.00000 0.00000 0.00000
- added joint jointfix_10_33: type fixed, parent link1_33, child left_lower_arm, origin xyz=0.00000 0.00000 0.00000 rpy=0.00000 -0.00000 0.00000, axis 0.00000 0.00000 0.00000
- added joint jointfix_11_31: type fixed, parent link1_31, child left_upper_arm, origin xyz=0.00000 0.00000 0.00000 rpy=0.00000 -0.00000 0.00000, axis 0.00000 0.00000 0.00000
- added joint jointfix_1_11: type fixed, parent link1_11, child right_shin, origin xyz=0.00000 0.00000 -0.02000 rpy=0.00000 -0.00000 0.00000, axis 0.00000 0.00000 0.00000
- added joint jointfix_2_9: type fixed, parent link1_9, child right_thigh, origin xyz=0.00000 0.00000 0.00000 rpy=0.00000 -0.00000 0.00000, axis 0.00000 0.00000 0.00000
- added joint jointfix_3_23: type fixed, parent link1_23, child left_foot, origin xyz=0.00000 0.00000 -0.08000 rpy=0.00000 -0.00000 0.00000, axis 0.00000 0.00000 0.00000
- added joint jointfix_4_20: type fixed, parent link1_20, child left_shin, origin xyz=0.00000 0.00000 -0.02000 rpy=0.00000 -0.00000 0.00000, axis 0.00000 0.00000 0.00000
- added joint jointfix_5_18: type fixed, parent link1_18, child left_thigh, origin xyz=0.00000 0.00000 0.00000 rpy=0.00000 -0.00000 0.00000, axis 0.00000 0.00000 0.00000
- added joint jointfix_6_5: type fixed, parent link1_5, child pelvis, origin xyz=0.00000 0.00000 -0.10000 rpy=0.00000 -0.00000 0.00000, axis 0.00000 0.00000 0.00000
- added joint jointfix_7_3: type fixed, parent link1_3, child lwaist, origin xyz=0.00000 0.00000 -0.06500 rpy=0.00000 -0.00000 0.00000, axis 0.00000 0.00000 0.00000
- added joint jointfix_8_28: type fixed, parent link1_28, child right_lower_arm, origin xyz=0.00000 0.00000 0.00000 rpy=0.00000 -0.00000 0.00000, axis 0.00000 0.00000 0.00000
- added joint jointfix_9_26: type fixed, parent link1_26, child right_upper_arm, origin xyz=0.00000 0.00000 0.00000 rpy=0.00000 -0.00000 0.00000, axis 0.00000 0.00000 0.00000
- added joint left_ankle_x: type continuous, parent link1_22, child link1_23, origin xyz=0.00000 0.00000 -0.04000 rpy=0.00000 -0.00000 0.00000, axis 1.00000 0.00000 0.50000
- added joint left_ankle_y: type continuous, parent left_shin, child link1_22, origin xyz=0.00000 0.00000 -0.31000 rpy=0.00000 -0.00000 0.00000, axis 0.00000 1.00000 0.00000
- added joint left_elbow: type continuous, parent left_upper_arm, child link1_33, origin xyz=0.18000 0.18000 -0.18000 rpy=0.00000 -0.00000 0.00000, axis 0.00000 -1.00000 -1.00000
- added joint left_hip_x: type continuous, parent pelvis, child link1_16, origin xyz=0.00000 0.10000 -0.04000 rpy=0.00000 -0.00000 0.00000, axis -1.00000 0.00000 0.00000
- added joint left_hip_y: type continuous, parent link1_17, child link1_18, origin xyz=0.00000 0.00000 0.00000 rpy=0.00000 -0.00000 0.00000, axis 0.00000 1.00000 0.00000
- added joint left_hip_z: type continuous, parent link1_16, child link1_17, origin xyz=0.00000 0.00000 0.00000 rpy=0.00000 -0.00000 0.00000, axis 0.00000 0.00000 -1.00000
- added joint left_knee: type continuous, parent left_thigh, child link1_20, origin xyz=0.00000 -0.01000 -0.38300 rpy=0.00000 -0.00000 0.00000, axis 0.00000 -1.00000 0.00000
- added joint left_shoulder1: type continuous, parent torso, child link1_30, origin xyz=0.00000 0.17000 0.06000 rpy=0.00000 -0.00000 0.00000, axis 2.00000 -1.00000 1.00000
- added joint left_shoulder2: type continuous, parent link1_30, child link1_31, origin xyz=0.00000 0.00000 0.00000 rpy=0.00000 -0.00000 0.00000, axis 0.00000 1.00000 1.00000
- added joint right_ankle_x: type continuous, parent link1_13, child link1_14, origin xyz=0.00000 0.00000 -0.04000 rpy=0.00000 -0.00000 0.00000, axis 1.00000 0.00000 0.50000
- added joint right_ankle_y: type continuous, parent right_shin, child link1_13, origin xyz=0.00000 0.00000 -0.31000 rpy=0.00000 -0.00000 0.00000, axis 0.00000 1.00000 0.00000
- added joint right_elbow: type continuous, parent right_upper_arm, child link1_28, origin xyz=0.18000 -0.18000 -0.18000 rpy=0.00000 -0.00000 0.00000, axis 0.00000 -1.00000 1.00000
- added joint right_hip_x: type continuous, parent pelvis, child link1_7, origin xyz=0.00000 -0.10000 -0.04000 rpy=0.00000 -0.00000 0.00000, axis 1.00000 0.00000 0.00000
- added joint right_hip_y: type continuous, parent link1_8, child link1_9, origin xyz=0.00000 0.00000 0.00000 rpy=0.00000 -0.00000 0.00000, axis 0.00000 1.00000 0.00000
- added joint right_hip_z: type continuous, parent link1_7, child link1_8, origin xyz=0.00000 0.00000 0.00000 rpy=0.00000 -0.00000 0.00000, axis 0.00000 0.00000 1.00000
- added joint right_knee: type continuous, parent right_thigh, child link1_11, origin xyz=0.00000 0.01000 -0.38300 rpy=0.00000 -0.00000 0.00000, axis 0.00000 -1.00000 0.00000
- added joint right_shoulder1: type continuous, parent torso, child link1_25, origin xyz=0.00000 -0.17000 0.06000 rpy=0.00000 -0.00000 0.00000, axis 2.00000 1.00000 1.00000
- added joint right_shoulder2: type continuous, parent link1_25, child link1_26, origin xyz=0.00000 0.00000 0.00000 rpy=0.00000 -0.00000 0.00000, axis 0.00000 -1.00000 1.00000
- joint BTy_joint: axis 0 1 0 -> 0.00000 1.00000 0.00000; child BTy_joint -> link1_3; limit lower=-0.349066 upper=0.349066 effort=100 velocity=1 -> (none); origin (none) -> xyz=0.00000 0.00000 0.00000 rpy=0.00000 -0.00000 0.00000; parent BTz_joint -> link1_2; type revolute -> continuous
- joint BTz_joint: axis 0 0 1 -> 0.00000 0.00000 1.00000; child BTz_joint -> link1_2; limit lower=-0.628319 upper=0.628319 effort=100 velocity=1 -> (none); origin (none) -> xyz=-0.01026 0.00000 -0.19500 rpy=0.00000 -0.00400 0.00000; parent BTx_joint -> torso; type revolute -> continuous
