Commit message: Add GPU acceleration to the Model in utils.py

File: data/objects/mmm.urdf (robot description, URDF)
Before this commit: robot Winter, 126 links, 125 joints
Links:
- removed link BLNsegment_joint
- removed link BLNx_joint
- removed link BLNy_joint
- removed link BLNz_joint
- removed link BPSegment_joint
- removed link BPx_joint
- removed link BPy_joint
- removed link BPz_joint
- removed link BTSegment_joint
- removed link BTx_joint
- removed link BTy_joint
- removed link BTz_joint
- removed link BUNsegment_joint
- removed link BUNx_joint
- removed link BUNy_joint
- removed link BUNz_joint
- removed link HeadSegment_joint
- removed link LAsegment_joint
- removed link LAx_joint
- removed link LAy_joint
- removed link LAz_joint
- removed link LEsegment_joint
- removed link LEx_joint
- removed link LEz_joint
- removed link LFx_joint
- removed link LHsegment_joint
- removed link LHx_joint
- removed link LHy_joint
- removed link LHz_joint
- removed link LKsegment_joint
- removed link LKx_joint
- removed link LMrot_joint
- removed link LSCsegment_joint
- removed link LSCx_joint
- removed link LSCy_joint
- removed link LSCz_joint
- removed link LSsegment_joint
- removed link LSx_joint
- removed link LSy_joint
- removed link LSz_joint
- removed link LWsegment_joint
- removed link LWx_joint
- removed link LWy_joint
- removed link LeftEyeSegmentX_joint
- removed link LeftEyeSegmentY_joint
- removed link LeftFingerJoint11y_joint
- removed link LeftFingerJoint11z_joint
- removed link LeftFingerJoint12y_joint
- removed link LeftFingerJoint13y_joint
- removed link LeftFingerJoint21x_joint
- removed link LeftFingerJoint21y_joint
- removed link LeftFingerJoint22y_joint
- removed link LeftFingerJoint23y_joint
- removed link LeftFingerJoint31x_joint
- removed link LeftFingerJoint31y_joint
- removed link LeftFingerJoint32y_joint
- removed link LeftFingerJoint33y_joint
- removed link LeftFingerJoint40y_joint
- removed link LeftFingerJoint41x_joint
- removed link LeftFingerJoint41y_joint
- removed link LeftFingerJoint42y_joint
- removed link LeftFingerJoint43y_joint
- removed link LeftFingerJoint50y_joint
- removed link LeftFingerJoint51x_joint
- removed link LeftFingerJoint51y_joint
- removed link LeftFingerJoint52y_joint
- removed link LeftFingerJoint53y_joint
- removed link LeftFootHeight_joint
- removed link LeftHandSegment_joint
- removed link MidHeadSegment_joint
- removed link RAsegment_joint
- removed link RAx_joint
- removed link RAy_joint
- removed link RAz_joint
- removed link REsegment_joint
- removed link REx_joint
- removed link REz_joint
- removed link RFx_joint
- removed link RHsegment_joint
- removed link RHx_joint
- removed link RHy_joint
- removed link RHz_joint
- removed link RKsegment_joint
- removed link RKx_joint
- removed link RMrot_joint
- removed link RSCsegment_joint
- removed link RSCx_joint
- removed link RSCy_joint
- removed link RSCz_joint
- removed link RSsegment_joint
- removed link RSx_joint
- removed link RSy_joint
- removed link RSz_joint
- removed link RWsegment_joint
- removed link RWx_joint
- removed link RWy_joint
- removed link RightEyeSegmentX_joint
- removed link RightEyeSegmentY_joint
- removed link RightFingerJoint11y_joint
- removed link RightFingerJoint11z_joint
- removed link RightFingerJoint12y_joint
- removed link RightFingerJoint13y_joint
- removed link RightFingerJoint21x_joint
- removed link RightFingerJoint21y_joint
- removed link RightFingerJoint22y_joint
- removed link RightFingerJoint23y_joint
- removed link RightFingerJoint31x_joint
- removed link RightFingerJoint31y_joint
- removed link RightFingerJoint32y_joint
- removed link RightFingerJoint33y_joint
- removed link RightFingerJoint40y_joint
- removed link RightFingerJoint41x_joint
- removed link RightFingerJoint41y_joint
- removed link RightFingerJoint42y_joint
- removed link RightFingerJoint43y_joint
- removed link RightFingerJoint50y_joint
- removed link RightFingerJoint51x_joint
- removed link RightFingerJoint51y_joint
- removed link RightFingerJoint52y_joint
- removed link RightFingerJoint53y_joint
- removed link RightFootHeight_joint
- removed link RightFootLength_joint
- removed link RightHandSegment_joint
- removed link collarSegment_joint
- removed link root
- removed link root_joint
- added link Head, mass 2.2392; collision sphere radius=0.089005; visual sphere radius=0.089005
- added link Head_f1, mass 0
- added link Head_f2, mass 0
- added link L3, mass 6.3444; collision box size=0.13815 0.16323 0.085916; visual box size=0.13815 0.16323 0.085916
- added link L3_f1, mass 0
- added link L3_f2, mass 0
- added link L5, mass 6.3444; collision box size=0.13815 0.16323 0.095104; visual box size=0.13815 0.16323 0.095104
- added link L5_f1, mass 0
- added link L5_f2, mass 0
- added link LeftFoot, mass 0.8086; collision box size=0.17983 0.074775 0.078509; visual box size=0.17983 0.074775 0.078509
- added link LeftFoot_f1, mass 0
- added link LeftFoot_f2, mass 0
- added link LeftForeArm, mass 1.244; collision cylinder length=0.22247 radius=0.019633; visual cylinder length=0.22247 radius=0.019633
- added link LeftForeArm_f1, mass 0
- added link LeftForeArm_f2, mass 0
- added link LeftHand, mass 0.3732; collision box size=0.11145 0.16718 0.039266; visual box size=0.11145 0.16718 0.039266
- added link LeftHandCOM, mass 0.00001; visual box size=0 0 0
- added link LeftHand_f1, mass 0
- added link LeftHand_f2, mass 0
- added link LeftLowerLeg, mass 2.2703; collision cylinder length=0.40608 radius=0.037388; visual cylinder length=0.40608 radius=0.037388
- added link LeftLowerLeg_f1, mass 0
- added link LeftLowerLeg_f2, mass 0
- added link LeftShoulder, mass 1.9282; collision cylinder length=0.13047 radius=0.023574; visual cylinder length=0.13047 radius=0.023574
- added link LeftShoulder_f1, mass 0
- added link LeftShoulder_f2, mass 0
- added link LeftToe, mass 0.0933; collision box size=0.060173 0.074775 0.014191; visual box size=0.060173 0.074775 0.014191
- added link LeftToe_f1, mass 0
- added link LeftToe_f2, mass 0
- added link LeftUpperArm, mass 1.866; collision cylinder length=0.26994 radius=0.029449; visual cylinder length=0.26994 radius=0.029449
- added link LeftUpperArm_f1, mass 0
- added link LeftUpperArm_f2, mass 0
- added link LeftUpperLeg, mass 7.775; collision cylinder length=0.44898 radius=0.0565; visual cylinder length=0.44898 radius=0.0565
- added link LeftUpperLeg_f1, mass 0
- added link LeftUpperLeg_f2, mass 0
- added link Neck, mass 0.7464; collision cylinder length=0.089252 radius=0.014205; visual cylinder length=0.089252 radius=0.014205
- added link Neck_f1, mass 0
- added link Neck_f2, mass 0
- added link Pelvis, mass 4.976; collision box size=0.13815 0.24914 0.097469; visual box size=0.13815 0.24914 0.097469
- added link RightFoot, mass 0.8086; collision box size=0.17983 0.074775 0.078509; visual box size=0.17983 0.074775 0.078509
- added link RightFoot_f1, mass 0
- added link RightFoot_f2, mass 0
- added link RightForeArm, mass 1.244; collision cylinder length=0.22247 radius=0.019633; visual cylinder length=0.22247 radius=0.019633
- added link RightForeArm_f1, mass 0
- added link RightForeArm_f2, mass 0
- added link RightHand, mass 0.3732; collision box size=0.11145 0.16718 0.039266; visual box size=0.11145 0.16718 0.039266
- added link RightHandCOM, mass 0.00001; visual box size=0 0 0
- added link RightHand_f1, mass 0
- added link RightHand_f2, mass 0
- added link RightLowerLeg, mass 2.2703; collision cylinder length=0.40608 radius=0.037388; visual cylinder length=0.40608 radius=0.037388
- added link RightLowerLeg_f1, mass 0
- added link RightLowerLeg_f2, mass 0
- added link RightShoulder, mass 1.9282; collision cylinder length=0.13047 radius=0.023574; visual cylinder length=0.13047 radius=0.023574
- added link RightShoulder_f1, mass 0
- added link RightShoulder_f2, mass 0
- added link RightToe, mass 0.0933; collision box size=0.060173 0.074775 0.014191; visual box size=0.060173 0.074775 0.014191
- added link RightToe_f1, mass 0
- added link RightToe_f2, mass 0
- added link RightUpperArm, mass 1.866; collision cylinder length=0.26994 radius=0.029449; visual cylinder length=0.26994 radius=0.029449
- added link RightUpperArm_f1, mass 0
- added link RightUpperArm_f2, mass 0
- added link RightUpperLeg, mass 7.775; collision cylinder length=0.44898 radius=0.0565; visual cylinder length=0.44898 radius=0.0565
- added link RightUpperLeg_f1, mass 0
- added link RightUpperLeg_f2, mass 0
- added link T12, mass 6.3444; collision box size=0.13815 0.16323 0.085916; visual box size=0.13815 0.16323 0.085916
- added link T12_f1, mass 0
- added link T12_f2, mass 0
- added link T8, mass 2.488; collision box size=0.13457 0.052626 0.11975; visual box size=0.13457 0.052626 0.11975
- added link T8_f1, mass 0
- added link T8_f2, mass 0
Joints:
- removed joint BLNsegment_joint
- removed joint BLNx_joint
- removed joint BLNy_joint
- removed joint BLNz_joint
- removed joint BPSegment_joint
- removed joint BPx_joint
- removed joint BPy_joint
- removed joint BPz_joint
- removed joint BTSegment_joint
- removed joint BTx_joint
- removed joint BTy_joint
- removed joint BTz_joint
- removed joint BUNsegment_joint
- removed joint BUNx_joint
- removed joint BUNy_joint
- removed joint BUNz_joint
- removed joint HeadSegment_joint
- removed joint LAsegment_joint
- removed joint LAx_joint
- removed joint LAy_joint
- removed joint LAz_joint
- removed joint LEsegment_joint
- removed joint LEx_joint
- removed joint LEz_joint
- removed joint LFx_joint
- removed joint LHsegment_joint
- removed joint LHx_joint
- removed joint LHy_joint
- removed joint LHz_joint
- removed joint LKsegment_joint
- removed joint LKx_joint
- removed joint LMrot_joint
- removed joint LSCsegment_joint
- removed joint LSCx_joint
- removed joint LSCy_joint
- removed joint LSCz_joint
- removed joint LSsegment_joint
- removed joint LSx_joint
- removed joint LSy_joint
- removed joint LSz_joint
- removed joint LWsegment_joint
- removed joint LWx_joint
- removed joint LWy_joint
- removed joint LeftEyeSegmentX_joint
- removed joint LeftEyeSegmentY_joint
- removed joint LeftFingerJoint11y_joint
- removed joint LeftFingerJoint11z_joint
- removed joint LeftFingerJoint12y_joint
- removed joint LeftFingerJoint13y_joint
- removed joint LeftFingerJoint21x_joint
- removed joint LeftFingerJoint21y_joint
- removed joint LeftFingerJoint22y_joint
- removed joint LeftFingerJoint23y_joint
- removed joint LeftFingerJoint31x_joint
- removed joint LeftFingerJoint31y_joint
- removed joint LeftFingerJoint32y_joint
- removed joint LeftFingerJoint33y_joint
- removed joint LeftFingerJoint40y_joint
- removed joint LeftFingerJoint41x_joint
- removed joint LeftFingerJoint41y_joint
- removed joint LeftFingerJoint42y_joint
- removed joint LeftFingerJoint43y_joint
- removed joint LeftFingerJoint50y_joint
- removed joint LeftFingerJoint51x_joint
- removed joint LeftFingerJoint51y_joint
- removed joint LeftFingerJoint52y_joint
- removed joint LeftFingerJoint53y_joint
- removed joint LeftFootHeight_joint
- removed joint LeftHandSegment_joint
- removed joint MidHeadSegment_joint
- removed joint RAsegment_joint
- removed joint RAx_joint
- removed joint RAy_joint
- removed joint RAz_joint
- removed joint REsegment_joint
- removed joint REx_joint
- removed joint REz_joint
- removed joint RFx_joint
- removed joint RHsegment_joint
- removed joint RHx_joint
- removed joint RHy_joint
- removed joint RHz_joint
- removed joint RKsegment_joint
- removed joint RKx_joint
- removed joint RMrot_joint
- removed joint RSCsegment_joint
- removed joint RSCx_joint
- removed joint RSCy_joint
- removed joint RSCz_joint
- removed joint RSsegment_joint
- removed joint RSx_joint
- removed joint RSy_joint
- removed joint RSz_joint
- removed joint RWsegment_joint
- removed joint RWx_joint
- removed joint RWy_joint
- removed joint RightEyeSegmentX_joint
- removed joint RightEyeSegmentY_joint
- removed joint RightFingerJoint11y_joint
- removed joint RightFingerJoint11z_joint
- removed joint RightFingerJoint12y_joint
- removed joint RightFingerJoint13y_joint
- removed joint RightFingerJoint21x_joint
- removed joint RightFingerJoint21y_joint
- removed joint RightFingerJoint22y_joint
- removed joint RightFingerJoint23y_joint
- removed joint RightFingerJoint31x_joint
- removed joint RightFingerJoint31y_joint
- removed joint RightFingerJoint32y_joint
- removed joint RightFingerJoint33y_joint
- removed joint RightFingerJoint40y_joint
- removed joint RightFingerJoint41x_joint
- removed joint RightFingerJoint41y_joint
- removed joint RightFingerJoint42y_joint
- removed joint RightFingerJoint43y_joint
- removed joint RightFingerJoint50y_joint
- removed joint RightFingerJoint51x_joint
- removed joint RightFingerJoint51y_joint
- removed joint RightFingerJoint52y_joint
- removed joint RightFingerJoint53y_joint
- removed joint RightFootHeight_joint
- removed joint RightFootLength_joint
- removed joint RightHandSegment_joint
- removed joint collarSegment_joint
- removed joint root_joint
- added joint jC1Head_rotx: type revolute, parent Neck, child Head_f1, origin xyz=0.000152           0    0.089252 rpy=0 0 0, axis 1 0 0, limit lower=-10.0 upper=10.0 effort=30 velocity=1.0
- added joint jC1Head_roty: type revolute, parent Head_f1, child Head_f2, origin xyz=0 0 0 rpy=0 0 0, axis 0 1 0, limit lower=-10.0 upper=10.0 effort=30 velocity=1.0
- added joint jC1Head_rotz: type revolute, parent Head_f2, child Head, origin xyz=0 0 0 rpy=0 0 0, axis 0 0 1, limit lower=-10.0 upper=10.0 effort=30 velocity=1.0
- added joint jL1T12_rotx: type revolute, parent L3, child T12_f1, origin xyz=0           0    0.085916 rpy=0 0 0, axis 1 0 0, limit lower=-10.0 upper=10.0 effort=30 velocity=1.0
- added joint jL1T12_roty: type revolute, parent T12_f1, child T12_f2, origin xyz=0 0 0 rpy=0 0 0, axis 0 1 0, limit lower=-10.0 upper=10.0 effort=30 velocity=1.0
- added joint jL1T12_rotz: type revolute, parent T12_f2, child T12, origin xyz=0 0 0 rpy=0 0 0, axis 0 0 1, limit lower=-10.0 upper=10.0 effort=30 velocity=1.0
- added joint jL4L3_rotx: type revolute, parent L5, child L3_f1, origin xyz=0.000374           0    0.095104 rpy=0 0 0, axis 1 0 0, limit lower=-10.0 upper=10.0 effort=30 velocity=1.0
- added joint jL4L3_roty: type revolute, parent L3_f1, child L3_f2, origin xyz=0 0 0 rpy=0 0 0, axis 0 1 0, limit lower=-10.0 upper=10.0 effort=30 velocity=1.0
- added joint jL4L3_rotz: type revolute, parent L3_f2, child L3, origin xyz=0 0 0 rpy=0 0 0, axis 0 0 1, limit lower=-10.0 upper=10.0 effort=30 velocity=1.0
- added joint jL5S1_rotx: type revolute, parent Pelvis, child L5_f1, origin xyz=-0.000206           0    0.098478 rpy=0 0 0, axis 1 0 0, limit lower=-10.0 upper=10.0 effort=30 velocity=1.0
- added joint jL5S1_roty: type revolute, parent L5_f1, child L5_f2, origin xyz=0 0 0 rpy=0 0 0, axis 0 1 0, limit lower=-10.0 upper=10.0 effort=30 velocity=1.0
- added joint jL5S1_rotz: type revolute, parent L5_f2, child L5, origin xyz=0 0 0 rpy=0 0 0, axis 0 0 1, limit lower=-10.0 upper=10.0 effort=30 velocity=1.0
- added joint jLeftAnkle_rotx: type revolute, parent LeftLowerLeg, child LeftFoot_f1, origin xyz=0.000205           0    -0.40608 rpy=0 0 0, axis 1 0 0, limit lower=-10.0 upper=10.0 effort=30 velocity=1.0
- added joint jLeftAnkle_roty: type revolute, parent LeftFoot_f1, child LeftFoot_f2, origin xyz=0 0 0 rpy=0 0 0, axis 0 1 0, limit lower=-10.0 upper=10.0 effort=30 velocity=1.0
- added joint jLeftAnkle_rotz: type revolute, parent LeftFoot_f2, child LeftFoot, origin xyz=0 0 0 rpy=0 0 0, axis 0 0 1, limit lower=-10.0 upper=10.0 effort=30 velocity=1.0
- added joint jLeftBallFoot_rotx: type revolute, parent LeftFoot, child LeftToe_f1, origin xyz=0.14456           0   -0.064752 rpy=0 0 0, axis 1 0 0, limit lower=-10.0 upper=10.0 effort=30 velocity=1.0
- added joint jLeftBallFoot_roty: type revolute, parent LeftToe_f1, child LeftToe_f2, origin xyz=0 0 0 rpy=0 0 0, axis 0 1 0, limit lower=-10.0 upper=10.0 effort=30 velocity=1.0
- added joint jLeftBallFoot_rotz: type revolute, parent LeftToe_f2, child LeftToe, origin xyz=0 0 0 rpy=0 0 0, axis 0 0 1, limit lower=-10.0 upper=10.0 effort=30 velocity=1.0
- added joint jLeftC7Shoulder_rotx: type revolute, parent T8, child LeftShoulder_f1, origin xyz=0    0.026313    0.067052 rpy=0 0 0, axis 1 0 0, limit lower=-10.0 upper=10.0 effort=30 velocity=1.0
- added joint jLeftC7Shoulder_roty: type revolute, parent LeftShoulder_f1, child LeftShoulder_f2, origin xyz=0 0 0 rpy=0 0 0, axis 0 1 0, limit lower=-10.0 upper=10.0 effort=30 velocity=1.0
- added joint jLeftC7Shoulder_rotz: type revolute, parent LeftShoulder_f2, child LeftShoulder, origin xyz=0 0 0 rpy=0 0 0, axis 0 0 1, limit lower=-10.0 upper=10.0 effort=30 velocity=1.0
- added joint jLeftElbow_rotx: type revolute, parent LeftUpperArm, child LeftForeArm_f1, origin xyz=0     0.26994           0 rpy=0 0 0, axis 1 0 0, limit lower=-10.0 upper=10.0 effort=30 velocity=1.0
- added joint jLeftElbow_roty: type revolute, parent LeftForeArm_f1, child LeftForeArm_f2, origin xyz=0 0 0 rpy=0 0 0, axis 0 1 0, limit lower=-10.0 upper=10.0 effort=30 velocity=1.0
- added joint jLeftElbow_rotz: type revolute, parent LeftForeArm_f2, child LeftForeArm, origin xyz=0 0 0 rpy=0 0 0, axis 0 0 1, limit lower=-10.0 upper=10.0 effort=30 velocity=1.0
- added joint jLeftHandCOM: type fixed, parent LeftHand, child LeftHandCOM, origin xyz=0 0.096206 0 rpy=0 0 0, axis 0 0 0
- added joint jLeftHip_rotx: type revolute, parent Pelvis, child LeftUpperLeg_f1, origin xyz=0.000103    0.081614    0.001009 rpy=0 0 0, axis 1 0 0, limit lower=-10.0 upper=10.0 effort=30 velocity=1.0
- added joint jLeftHip_roty: type revolute, parent LeftUpperLeg_f1, child LeftUpperLeg_f2, origin xyz=0 0 0 rpy=0 0 0, axis 0 1 0, limit lower=-10.0 upper=10.0 effort=30 velocity=1.0
- added joint jLeftHip_rotz: type revolute, parent LeftUpperLeg_f2, child LeftUpperLeg, origin xyz=0 0 0 rpy=0 0 0, axis 0 0 1, limit lower=-10.0 upper=10.0 effort=30 velocity=1.0
- added joint jLeftKnee_rotx: type revolute, parent LeftUpperLeg, child LeftLowerLeg_f1, origin xyz=3.6e-05           0    -0.44898 rpy=0 0 0, axis 1 0 0, limit lower=-10.0 upper=10.0 effort=30 velocity=1.0
- added joint jLeftKnee_roty: type revolute, parent LeftLowerLeg_f1, child LeftLowerLeg_f2, origin xyz=0 0 0 rpy=0 0 0, axis 0 1 0, limit lower=-10.0 upper=10.0 effort=30 velocity=1.0
- added joint jLeftKnee_rotz: type revolute, parent LeftLowerLeg_f2, child LeftLowerLeg, origin xyz=0 0 0 rpy=0 0 0, axis 0 0 1, limit lower=-10.0 upper=10.0 effort=30 velocity=1.0
- added joint jLeftShoulder_rotx: type revolute, parent LeftShoulder, child LeftUpperArm_f1, origin xyz=0     0.13047           0 rpy=0 0 0, axis 1 0 0, limit lower=-10.0 upper=10.0 effort=30 velocity=1.0
- added joint jLeftShoulder_roty: type revolute, parent LeftUpperArm_f1, child LeftUpperArm_f2, origin xyz=0 0 0 rpy=0 0 0, axis 0 1 0, limit lower=-10.0 upper=10.0 effort=30 velocity=1.0
- added joint jLeftShoulder_rotz: type revolute, parent LeftUpperArm_f2, child LeftUpperArm, origin xyz=0 0 0 rpy=0 0 0, axis 0 0 1, limit lower=-10.0 upper=10.0 effort=30 velocity=1.0
- added joint jLeftWrist_rotx: type revolute, parent LeftForeArm, child LeftHand_f1, origin xyz=7.7e-05     0.22247           0 rpy=0 0 0, axis 1 0 0, limit lower=-10.0 upper=10.0 effort=30 velocity=1.0
- added joint jLeftWrist_roty: type revolute, parent LeftHand_f1, child LeftHand_f2, origin xyz=0 0 0 rpy=0 0 0, axis 0 1 0, limit lower=-10.0 upper=10.0 effort=30 velocity=1.0
- added joint jLeftWrist_rotz: type revolute, parent LeftHand_f2, child LeftHand, origin xyz=0 0 0 rpy=0 0 0, axis 0 0 1, limit lower=-10.0 upper=10.0 effort=30 velocity=1.0
- added joint jRightAnkle_rotx: type revolute, parent RightLowerLeg, child RightFoot_f1, origin xyz=0.000205           0    -0.40608 rpy=0 0 0, axis 1 0 0, limit lower=-10.0 upper=10.0 effort=30 velocity=1.0
- added joint jRightAnkle_roty: type revolute, parent RightFoot_f1, child RightFoot_f2, origin xyz=0 0 0 rpy=0 0 0, axis 0 1 0, limit lower=-10.0 upper=10.0 effort=30 velocity=1.0
- added joint jRightAnkle_rotz: type revolute, parent RightFoot_f2, child RightFoot, origin xyz=0 0 0 rpy=0 0 0, axis 0 0 1, limit lower=-10.0 upper=10.0 effort=30 velocity=1.0
- added joint jRightBallFoot_rotx: type revolute, parent RightFoot, child RightToe_f1, origin xyz=0.14456           0   -0.064752 rpy=0 0 0, axis 1 0 0, limit lower=-10.0 upper=10.0 effort=30 velocity=1.0
- added joint jRightBallFoot_roty: type revolute, parent RightToe_f1, child RightToe_f2, origin xyz=0 0 0 rpy=0 0 0, axis 0 1 0, limit lower=-10.0 upper=10.0 effort=30 velocity=1.0
- added joint jRightBallFoot_rotz: type revolute, parent RightToe_f2, child RightToe, origin xyz=0 0 0 rpy=0 0 0, axis 0 0 1, limit lower=-10.0 upper=10.0 effort=30 velocity=1.0
- added joint jRightC7Shoulder_rotx: type revolute, parent T8, child RightShoulder_f1, origin xyz=0   -0.026313    0.067052 rpy=0 0 0, axis 1 0 0, limit lower=-10.0 upper=10.0 effort=30 velocity=1.0
- added joint jRightC7Shoulder_roty: type revolute, parent RightShoulder_f1, child RightShoulder_f2, origin xyz=0 0 0 rpy=0 0 0, axis 0 1 0, limit lower=-10.0 upper=10.0 effort=30 velocity=1.0
- added joint jRightC7Shoulder_rotz: type revolute, parent RightShoulder_f2, child RightShoulder, origin xyz=0 0 0 rpy=0 0 0, axis 0 0 1, limit lower=-10.0 upper=10.0 effort=30 velocity=1.0
- added joint jRightElbow_rotx: type revolute, parent RightUpperArm, child RightForeArm_f1, origin xyz=0    -0.26994           0 rpy=0 0 0, axis 1 0 0, limit lower=-10.0 upper=10.0 effort=30 velocity=1.0
- added joint jRightElbow_roty: type revolute, parent RightForeArm_f1, child RightForeArm_f2, origin xyz=0 0 0 rpy=0 0 0, axis 0 1 0, limit lower=-10.0 upper=10.0 effort=30 velocity=1.0
- added joint jRightElbow_rotz: type revolute, parent RightForeArm_f2, child RightForeArm, origin xyz=0 0 0 rpy=0 0 0, axis 0 0 1, limit lower=-10.0 upper=10.0 effort=30 velocity=1.0
- added joint jRightHandCOM: type fixed, parent RightHand, child RightHandCOM, origin xyz=0 -0.096206 0 rpy=0 0 0, axis 0 0 0
- added joint jRightHip_rotx: type revolute, parent Pelvis, child RightUpperLeg_f1, origin xyz=0.000103   -0.081614    0.001009 rpy=0 0 0, axis 1 0 0, limit lower=-10.0 upper=10.0 effort=30 velocity=1.0
- added joint jRightHip_roty: type revolute, parent RightUpperLeg_f1, child RightUpperLeg_f2, origin xyz=0 0 0 rpy=0 0 0, axis 0 1 0, limit lower=-10.0 upper=10.0 effort=30 velocity=1.0
- added joint jRightHip_rotz: type revolute, parent RightUpperLeg_f2, child RightUpperLeg, origin xyz=0 0 0 rpy=0 0 0, axis 0 0 1, limit lower=-10.0 upper=10.0 effort=30 velocity=1.0
- added joint jRightKnee_rotx: type revolute, parent RightUpperLeg, child RightLowerLeg_f1, origin xyz=3.6e-05           0    -0.44898 rpy=0 0 0, axis 1 0 0, limit lower=-10.0 upper=10.0 effort=30 velocity=1.0
- added joint jRightKnee_roty: type revolute, parent RightLowerLeg_f1, child RightLowerLeg_f2, origin xyz=0 0 0 rpy=0 0 0, axis 0 1 0, limit lower=-10.0 upper=10.0 effort=30 velocity=1.0
- added joint jRightKnee_rotz: type revolute, parent RightLowerLeg_f2, child RightLowerLeg, origin xyz=0 0 0 rpy=0 0 0, axis 0 0 1, limit lower=-10.0 upper=10.0 effort=30 velocity=1.0
- added joint jRightShoulder_rotx: type revolute, parent RightShoulder, child RightUpperArm_f1, origin xyz=0    -0.13047           0 rpy=0 0 0, axis 1 0 0, limit lower=-10.0 upper=10.0 effort=30 velocity=1.0
- added joint jRightShoulder_roty: type revolute, parent RightUpperArm_f1, child RightUpperArm_f2, origin xyz=0 0 0 rpy=0 0 0, axis 0 1 0, limit lower=-10.0 upper=10.0 effort=30 velocity=1.0
- added joint jRightShoulder_rotz: type revolute, parent RightUpperArm_f2, child RightUpperArm, origin xyz=0 0 0 rpy=0 0 0, axis 0 0 1, limit lower=-10.0 upper=10.0 effort=30 velocity=1.0
- added joint jRightWrist_rotx: type revolute, parent RightForeArm, child RightHand_f1, origin xyz=7.7e-05    -0.22247           0 rpy=0 0 0, axis 1 0 0, limit lower=-10.0 upper=10.0 effort=30 velocity=1.0
- added joint jRightWrist_roty: type revolute, parent RightHand_f1, child RightHand_f2, origin xyz=0 0 0 rpy=0 0 0, axis 0 1 0, limit lower=-10.0 upper=10.0 effort=30 velocity=1.0
- added joint jRightWrist_rotz: type revolute, parent RightHand_f2, child RightHand, origin xyz=0 0 0 rpy=0 0 0, axis 0 0 1, limit lower=-10.0 upper=10.0 effort=30 velocity=1.0
- added joint jT1C7_rotx: type revolute, parent T8, child Neck_f1, origin xyz=0           0     0.11975 rpy=0 0 0, axis 1 0 0, limit lower=-10.0 upper=10.0 effort=30 velocity=1.0
- added joint jT1C7_roty: type revolute, parent Neck_f1, child Neck_f2, origin xyz=0 0 0 rpy=0 0 0, axis 0 1 0, limit lower=-10.0 upper=10.0 effort=30 velocity=1.0
- added joint jT1C7_rotz: type revolute, parent Neck_f2, child Neck, origin xyz=0 0 0 rpy=0 0 0, axis 0 0 1, limit lower=-10.0 upper=10.0 effort=30 velocity=1.0
- added joint jT9T8_rotx: type revolute, parent T12, child T8_f1, origin xyz=0           0    0.085916 rpy=0 0 0, axis 1 0 0, limit lower=-10.0 upper=10.0 effort=30 velocity=1.0
- added joint jT9T8_roty: type revolute, parent T8_f1, child T8_f2, origin xyz=0 0 0 rpy=0 0 0, axis 0 1 0, limit lower=-10.0 upper=10.0 effort=30 velocity=1.0
- added joint jT9T8_rotz: type revolute, parent T8_f2, child T8, origin xyz=0 0 0 rpy=0 0 0, axis 0 0 1, limit lower=-10.0 upper=10.0 effort=30 velocity=1.0
